File: Electronic/EAGLE/board-beta.0.2.brd (EAGLE design)
At the start: 69.5 x 57.1 mm, 23 parts, among them CN2 1X4SMT, J1 JACK2.1MM, Q1 IRF630N, Q3 IRF9Z34, Q4 IRF9734, Q5 IRFZ44, Q6 IRFZ44, Q7 IRF630N, Q8 BD139

Commit message: nueva vetrsion
Parts:
- added FAN2: 1X4SMT, adafruit:1X4-SMT
- moved Q8 93.8 mm to (55.9, 45.9), turned to 180 degrees
- moved R2 87.0 mm to (48.6, 47.1)
- moved CN2 5.59 mm to (60.8, 37.1)
- moved R9 2.00 mm to (43.7, 47.1)
Connections:
- removed net N$23: U$1.VIN
- net VCC_12V: now also U$1.VIN
Routing:
- net VCC_12V: track 128.7 -> 167.7 mm
- net D3: track 0.00 -> 12.3 mm
- net D0: track 6.88 -> 14.9 mm
- net FAN_1: track 20.9 -> 14.8 mm
- net LED_1: track 19.4 -> 13.2 mm
- net N$11: track 0.00 -> 3.39 mm
- net D9: track 7.87 -> 5.87 mm
- net N$12: track 5.48 -> 7.03 mm
- net GND: track 153.3 -> 152.0 mm
- net D5: track 18.3 -> 17.2 mm
Changed lines of the file:
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@@
 <setting verticaltext="up"/>
 </settings>
-<grid distance="0.1" unitdist="mm" unit="mm" style="lines" multiple="1" display="yes" altdistance="0.025" altunitdist="inch" altunit="inch"/>
+<grid distance="0.05" unitdist="inch" unit="inch" style="lines" multiple="1" display="no" altdistance="0.025" altunitdist="inch" altunit="inch"/>
 <layers>
 <layer number="1" name="Top" color="4" fill="1" visible="yes" active="yes"/>
@@
 </autorouter>
 <elements>
-<element name="CN2" library="adafruit" package="1X4-SMT" value="1X4SMT" x="63.45" y="42.02" rot="R270"/>
+<element name="CN2" library="adafruit" package="1X4-SMT" value="1X4SMT" x="60.75" y="37.12" rot="R270"/>
 <element name="H+T" library="adafruit" package="1X4-SMT" value="1X4SMT" x="63.45" y="12.81" rot="R90"/>
 <element name="J1" library="fab" package="JACK_2.1MM" value="JACK2.1MM" x="6.3" y="10.27" rot="R270"/>
@@
 <element name="R7" library="fab" package="R1206FAB" value="1k" x="8.84" y="41.48" rot="R270"/>
 <element name="R8" library="fab" package="R1206FAB" value="0" x="45.57" y="15.35" rot="R180"/>
-<element name="R9" library="fab" package="R1206FAB" value="1k" x="45.67" y="47.1"/>
+<element name="R9" library="fab" package="R1206FAB" value="1k" x="43.67" y="47.1"/>
 <element name="U$1" library="adafruit" package="ARDUINO" value="ARDUINOUNO" x="1.22" y="1.38"/>
 <element name="JP1" library="fab" package="2X03SMD" value="" x="63.75" y="26.82"/>
-<element name="R2" library="fab" package="R1206FAB" value="1k" x="-2.9" y="-23"/>
-<element name="Q8" library="transistor-power" package="TO126AV" value="BD139" x="4.6" y="-32.6"/>
+<element name="R2" library="fab" package="R1206FAB" value="1k" x="48.6" y="47.1"/>
+<element name="Q8" library="transistor-power" package="TO126AV" value="BD139" x="55.9" y="45.9" rot="R180"/>
+<element name="FAN2" library="adafruit" package="1X4-SMT" value="1X4SMT" x="0" y="-8.89"/>
 </elements>
 <signals>
@@
 <contactref element="U$1" pad="D0"/>
 <contactref element="CN2" pad="1"/>
-<wire x1="63.45" y1="45.83" x2="63.45" y2="50.91" width="0.4064" layer="1"/>
-<wire x1="63.45" y1="50.91" x2="64.72" y2="52.18" width="0.4064" layer="1"/>
+<wire x1="64.72" y1="52.18" x2="64.72" y2="41.86" width="0.4064" layer="1"/>
+<wire x1="64.72" y1="41.86" x2="63.5" y2="40.64" width="0.4064" layer="1"/>
+<wire x1="63.5" y1="40.64" x2="61.04" y2="40.64" width="0.4064" layer="1"/>
+<wire x1="61.04" y1="40.64" x2="60.75" y2="40.93" width="0.4064" layer="1"/>
 </signal>
 <signal name="D1">
@@
 <contactref element="R6" pad="1"/>
 <contactref element="U$1" pad="D5"/>
-<wire x1="41.86" y1="42.401" x2="44.601" y2="42.401" width="0.4064" layer="1"/>
-<wire x1="44.601" y1="42.401" x2="45.5" y2="43.3" width="0.4064" layer="1"/>
-<wire x1="45.5" y1="43.3" x2="45.5" y2="48.3" width="0.4064" layer="1"/>
-<wire x1="45.5" y1="48.3" x2="46.6" y2="49.4" width="0.4064" layer="1"/>
-<wire x1="46.6" y1="49.4" x2="51.1" y2="49.4" width="0.4064" layer="1"/>
-<wire x1="51.1" y1="49.4" x2="52.1" y2="50.4" width="0.4064" layer="1"/>
-<wire x1="52.1" y1="50.4" x2="52.1" y2="52.1" width="0.4064" layer="1"/>
+<wire x1="41.86" y1="42.401" x2="41.901" y2="42.401" width="0.4064" layer="1"/>
+<wire x1="41.901" y1="42.401" x2="43.6" y2="43.9" width="0.4064" layer="1"/>
+<wire x1="43.6" y1="43.9" x2="43.6" y2="48.8" width="0.4064" layer="1"/>
+<wire x1="43.6" y1="48.8" x2="45.2" y2="50.4" width="0.4064" layer="1"/>
+<wire x1="45.2" y1="50.4" x2="50.3" y2="50.4" width="0.4064" layer="1"/>
+<wire x1="50.3" y1="50.4" x2="52.1" y2="52.1" width="0.4064" layer="1"/>
 <wire x1="52.1" y1="52.1" x2="52.02" y2="52.18" width="0.4064" layer="1"/>
 </signal>
@@
 <contactref element="U$1" pad="A1"/>
 </signal>
-<signal name="N$23">
-<contactref element="U$1" pad="VIN"/>
-</signal>
 <signal name="N$24">
 <contactref element="U$1" pad="GND1"/>
@@
 <wire x1="4.3188" y1="15.9088" x2="6.3" y2="17.89" width="1.27" layer="1"/>
 <wire x1="6.3" y1="17.89" x2="16.46" y2="17.89" width="1.27" layer="1"/>
-<wire x1="30.43" y1="17.89" x2="30.43" y2="2.65" width="0.4064" layer="1"/>
-<wire x1="30.43" y1="2.65" x2="31.7" y2="1.38" width="0.4064" layer="1"/>
-<wire x1="31.7" y1="1.38" x2="40.59" y2="1.38" width="0.4064" layer="1"/>
-<wire x1="40.59" y1="1.38" x2="41.86" y2="2.65" width="0.4064" layer="1"/>
+<wire x1="30.43" y1="17.89" x2="30.43" y2="3.85" width="0.4064" layer="1"/>
+<wire x1="30.43" y1="3.85" x2="31.5" y2="2.28" width="0.4064" layer="1"/>
+<wire x1="31.5" y1="2.28" x2="41.49" y2="2.28" width="0.4064" layer="1"/>
+<wire x1="41.49" y1="2.28" x2="41.86" y2="2.65" width="0.4064" layer="1"/>
 <wire x1="41.86" y1="2.65" x2="41.86" y2="3.92" width="0.4064" layer="1"/>
 <wire x1="16.46" y1="17.89" x2="22.81" y2="17.89" width="1.27" layer="1"/>
@@
 <contactref element="Q8" pad="C"/>
 <wire x1="53.29" y1="14.08" x2="51.639" y2="28.05" width="0" layer="19" extent="1-1"/>
-<wire x1="4.6" y1="-33.87" x2="31.7" y2="1.38" width="0" layer="19" extent="1-1"/>
+<wire x1="55.9" y1="47.17" x2="31.5" y2="2.28" width="0" layer="19" extent="1-1"/>
 </signal>
 <signal name="VCC_12V">
@@
 <wire x1="57.1" y1="21.7" x2="57.1" y2="25.51" width="1.27" layer="1"/>
 <wire x1="57.1" y1="25.51" x2="57.1" y2="30.59" width="1.27" layer="16"/>
-<wire x1="57.1" y1="30.59" x2="57.1" y2="36.686" width="1.27" layer="1"/>
-<wire x1="57.1" y1="36.686" x2="58.624" y2="38.21" width="1.27" layer="1"/>
-<wire x1="58.624" y1="38.21" x2="63.45" y2="38.21" width="1.27" layer="1"/>
+<wire x1="57.1" y1="30.59" x2="57.1" y2="31.786" width="1.27" layer="1"/>
+<wire x1="57.1" y1="31.786" x2="58.624" y2="33.31" width="1.27" layer="1"/>
+<wire x1="58.624" y1="33.31" x2="60.75" y2="33.31" width="1.27" layer="1"/>
 <via x="31.7" y="32.114" extent="1-16" drill="0.8" shape="octagon"/>
 <via x="38.812" y="32.114" extent="1-16" drill="0.8" shape="octagon"/>
 <via x="57.1" y="30.59" extent="1-16" drill="0.8" shape="octagon"/>
 <via x="57.1" y="25.51" extent="1-16" drill="0.8" shape="octagon"/>
+<contactref element="U$1" pad="VIN"/>
+<wire x1="46.94" y1="3.92" x2="46.94" y2="2.64" width="1.27" layer="1"/>
+<wire x1="46.94" y1="2.64" x2="45.2" y2="0.9" width="1.27" layer="1"/>
+<wire x1="45.2" y1="0.9" x2="7.4912" y2="0.9" width="1.27" layer="1"/>
+<wire x1="7.4912" y1="0.9" x2="3.887" y2="4.5042" width="1.27" layer="1"/>
 </signal>
 <signal name="D10">
@@
 <contactref element="CN2" pad="2"/>
 <contactref element="Q7" pad="3"/>
-<wire x1="63.45" y1="43.29" x2="54.56" y2="43.29" width="1.27" layer="1"/>
-<wire x1="54.56" y1="43.29" x2="52.02" y2="40.75" width="1.27" layer="1"/>
-<wire x1="52.02" y1="40.75" x2="52.02" y2="38.21" width="1.27" layer="1"/>
-<wire x1="52.02" y1="38.21" x2="50.75" y2="36.94" width="1.27" layer="1"/>
-<wire x1="50.75" y1="36.94" x2="48.21" y2="36.94" width="1.27" layer="1"/>
+<wire x1="60.75" y1="38.39" x2="51.09" y2="38.39" width="1.27" layer="1"/>
+<wire x1="51.09" y1="38.39" x2="49.53" y2="36.83" width="1.27" layer="1"/>
+<wire x1="49.53" y1="36.83" x2="48.32" y2="36.83" width="1.27" layer="1"/>
+<wire x1="48.32" y1="36.83" x2="48.21" y2="36.94" width="1.27" layer="1"/>
 </signal>
 <signal name="D3">
 <contactref element="R2" pad="1"/>
 <contactref element="U$1" pad="D3"/>
-<wire x1="-4.551" y1="-23" x2="57.1" y2="52.18" width="0" layer="19" extent="1-1"/>
+<wire x1="46.949" y1="47.1" x2="48.5" y2="48.9" width="0.4064" layer="1"/>
+<wire x1="48.5" y1="48.9" x2="49" y2="49.5" width="0.4064" layer="1"/>
+<wire x1="49" y1="49.5" x2="54.2" y2="49.5" width="0.4064" layer="1"/>
+<wire x1="54.2" y1="49.5" x2="55.62" y2="50.8" width="0.4064" layer="1"/>
+<wire x1="55.62" y1="50.8" x2="57.1" y2="52.18" width="0.4064" layer="1"/>
 </signal>
 <signal name="FAN_1">
 <contactref element="CN2" pad="3"/>
 <contactref element="Q1" pad="3"/>
-<wire x1="63.45" y1="40.75" x2="55.83" y2="40.75" width="1.27" layer="1"/>
-<wire x1="55.83" y1="40.75" x2="54.56" y2="39.48" width="1.27" layer="1"/>
-<wire x1="54.56" y1="39.48" x2="54.56" y2="36.94" width="1.27" layer="1"/>
-<wire x1="54.56" y1="36.94" x2="48.21" y2="30.59" width="1.27" layer="1"/>
+<wire x1="60.75" y1="35.85" x2="54.9" y2="35.85" width="1.27" layer="1"/>
+<wire x1="54.9" y1="35.85" x2="49.53" y2="30.48" width="1.27" layer="1"/>
+<wire x1="49.53" y1="30.48" x2="48.32" y2="30.48" width="1.27" layer="1"/>
+<wire x1="48.32" y1="30.48" x2="48.21" y2="30.59" width="1.27" layer="1"/>
 </signal>
 <signal name="N$4">
@@
 <contactref element="R9" pad="2"/>
 <contactref element="Q7" pad="1"/>
-<wire x1="47.321" y1="47.1" x2="47.3" y2="47.1" width="0.4064" layer="1"/>
-<wire x1="47.3" y1="47.1" x2="47.3" y2="42.93" width="0.4064" layer="1"/>
-<wire x1="47.3" y1="42.93" x2="48.21" y2="42.02" width="0.4064" layer="1"/>
+<wire x1="45.321" y1="47.1" x2="45.3" y2="43.8" width="0.4064" layer="1"/>
+<wire x1="45.3" y1="43.8" x2="46.8" y2="42.03" width="0.4064" layer="1"/>
+<wire x1="46.8" y1="42.03" x2="48.21" y2="42.02" width="0.4064" layer="1"/>
 </signal>
 <signal name="N$2">
@@
 <contactref element="R2" pad="2"/>
 <contactref element="Q8" pad="B"/>
-<wire x1="-1.249" y1="-23" x2="6.886" y2="-33.87" width="0" layer="19" extent="1-1"/>
+<wire x1="50.251" y1="47.1" x2="53.544" y2="47.1" width="0.4064" layer="1"/>
+<wire x1="53.544" y1="47.1" x2="53.614" y2="47.17" width="0.4064" layer="1"/>
 </signal>
 <signal name="D9">
@@
 <wire x1="40.336" y1="52.18" x2="40.336" y2="48.624" width="0.4064" layer="1"/>
 <wire x1="40.336" y1="48.624" x2="41.86" y2="47.1" width="0.4064" layer="1"/>
-<wire x1="41.86" y1="47.1" x2="44.019" y2="47.1" width="0.4064" layer="1"/>
+<wire x1="41.86" y1="47.1" x2="42.019" y2="47.1" width="0.4064" layer="1"/>
 </signal>
 <signal name="FAN_2">
