File: Electronic/EAGLE/board-beta.0.2.sch (EAGLE design)
At the start: 23 parts, among them CN2 1X4SMT, J1 JACK2.1MM, Q1 IRF630N, Q3 IRF9Z34, Q4 IRF9734, Q5 IRFZ44, Q6 IRFZ44, Q7 IRF630N, Q8 BD139

Commit message: nueva vetrsion
Parts:
- added FAN2: 1X4SMT, adafruit:1X4SMT
Connections:
- removed net N$23: U$1.VIN
- new net FAN_2: Q8.E
- net LED_1: no longer Q8.E
- net VCC_12V: now also U$1.VIN
Changed lines of the file:
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@@
 <part name="GND4" library="supply1" deviceset="GND" device=""/>
 <part name="Q8" library="transistor-power" deviceset="BD139" device=""/>
+<part name="FAN2" library="adafruit" deviceset="1X4" device="SMT"/>
 </parts>
 <sheets>
@@
 <instance part="GND4" gate="1" x="78.74" y="53.34" rot="R180"/>
 <instance part="Q8" gate="1" x="76.2" y="45.72"/>
+<instance part="FAN2" gate="G$1" x="-93.98" y="-40.64" rot="R180"/>
 </instances>
 <busses>
@@
 </segment>
 </net>
-<net name="N$23" class="0">
-<segment>
-<pinref part="U$1" gate="G$1" pin="VIN"/>
-<wire x1="-12.7" y1="5.08" x2="-12.7" y2="2.54" width="0.1524" layer="91"/>
-</segment>
-</net>
 <net name="N$24" class="0">
 <segment>
@@
 <wire x1="68.58" y1="25.4" x2="68.58" y2="27.94" width="0.1524" layer="91"/>
 <label x="68.58" y="27.94" size="1.778" layer="95" xref="yes"/>
+</segment>
+<segment>
+<pinref part="U$1" gate="G$1" pin="VIN"/>
+<wire x1="-12.7" y1="5.08" x2="-12.7" y2="2.54" width="0.1524" layer="91"/>
+<label x="-12.7" y="0" size="1.778" layer="95" rot="R270" xref="yes"/>
 </segment>
 </net>
@@
 <label x="81.28" y="58.42" size="1.778" layer="95" xref="yes"/>
 </segment>
-<segment>
-<wire x1="78.74" y1="40.64" x2="78.74" y2="35.56" width="0.1524" layer="91"/>
-<label x="81.28" y="35.56" size="1.778" layer="95" xref="yes"/>
-<pinref part="Q8" gate="1" pin="E"/>
-</segment>
 </net>
 <net name="D3" class="0">
@@
 </segment>
 </net>
+<net name="FAN_2" class="0">
+<segment>
+<wire x1="78.74" y1="40.64" x2="78.74" y2="35.56" width="0.1524" layer="91"/>
+<label x="81.28" y="35.56" size="1.778" layer="95" xref="yes"/>
+<pinref part="Q8" gate="1" pin="E"/>
+</segment>
+</net>
