File: Electronic/EAGLE/board-beta.0.2.sch (EAGLE design)
At the start: 24 parts, among them CN2 1X4SMT, J1 JACK2.1MM, Q1 IRF630N, Q2 IRF630N, Q3 IRF9Z34, Q4 IRF9734, Q5 IRFZ44, Q6 IRFZ44, Q7 IRF630N

Commit message: version Pi
Changed lines of the file:
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@@
 <text x="93.98" y="76.2" size="1.778" layer="91">Neg.</text>
 <text x="93.98" y="96.52" size="1.778" layer="91">Neg.</text>
+<wire x1="-53.34" y1="119.38" x2="-53.34" y2="-48.26" width="0.6096" layer="94" style="shortdash"/>
+<wire x1="22.86" y1="119.38" x2="22.86" y2="104.14" width="0.6096" layer="94" style="shortdash"/>
+<wire x1="22.86" y1="104.14" x2="22.86" y2="78.74" width="0.6096" layer="94" style="shortdash"/>
+<wire x1="22.86" y1="78.74" x2="22.86" y2="55.88" width="0.6096" layer="94" style="shortdash"/>
+<wire x1="22.86" y1="55.88" x2="22.86" y2="30.48" width="0.6096" layer="94" style="shortdash"/>
+<wire x1="22.86" y1="30.48" x2="22.86" y2="-48.26" width="0.6096" layer="94" style="shortdash"/>
+<wire x1="22.86" y1="78.74" x2="124.46" y2="78.74" width="0.6096" layer="94" style="shortdash"/>
+<wire x1="22.86" y1="55.88" x2="124.46" y2="55.88" width="0.6096" layer="94" style="shortdash"/>
+<wire x1="22.86" y1="30.48" x2="124.46" y2="30.48" width="0.6096" layer="94" style="shortdash"/>
+<wire x1="22.86" y1="104.14" x2="124.46" y2="104.14" width="0.6096" layer="94" style="shortdash"/>
 </plain>
 <instances>
