File: Electronic/EAGLE/board-beta.0.7.sch (EAGLE design)
At the start: 24 parts, among them CN2 1X4SMT, J1 JACK2.1MM, Q1 IRF630N, Q2 IRF630N, Q3 IRF9Z34, Q4 IRF9734, Q5 IRFZ44, Q6 IRFZ44, Q7 IRF630N

Commit message: version Pi
Parts:
- added D1, D2: (no value), fab:DIODESOD123
- CN2, H+T, LCD: value 1X4SMT -> (none); device adafruit:1X4SMT -> pinhead:PINHD-1X4
- FAN2: value 1X4SMT -> (none); device adafruit:1X4SMT -> con-lstb:MA04-1
- PELTIER: value 1X4SMT -> (none); device adafruit:1X4SMT -> pinhead:PINHD-1X2
Connections:
- net FAN_1: now also D2.A
- net FAN_2: now also D1.A
- net GND: now also J1.CONTACT; no longer J1.PIN, PELTIER.1
- net PEL_1: now also PELTIER.2; no longer PELTIER.3
- net PEL_2: now also PELTIER.1; no longer PELTIER.2
- net VCC_12V: now also D1.C, D2.C, J1.PIN; no longer J1.CONTACT, PELTIER.4
Other:
- note added: "-"
- note added: "A4950ELJTR-T A3950SLP-T"
- note added: "A4953(FabLab)"
- note added: "BD6231F-E2 BD6222FP-E2"
- note added: "Esteban Martin Gimenez"
- note added: "Microcosm Terraformation Module"
- note added: "PUMP"
- note added: "VALVULA"
- note added: "Version 0.7.1"
- note removed: "Neg."
- note removed: "Pump"
- note removed: "valvula"
