File: Electronic/EAGLE/schematic0.1v.brd (EAGLE design)
At the start: 68.5 x 56.4 mm, 14 parts, among them CN2 1X4SMT, CN3 1X4SMT, J1 JACK2.1MM

Commit message: nueva version Pi
Connections:
- net PEL_2: now also PELTIER.4; no longer PELTIER.2
- net VCC_12V: now also PELTIER.2; no longer PELTIER.4
Routing:
- net PEL_2: track 33.8 -> 21.0 mm
- net PEL_1: track 29.3 -> 21.0 mm
- net VCC_5V: track 69.9 -> 72.4 mm
- net VCC_12V: track 97.8 -> 96.3 mm, vias 4 -> 6
- net GND1: track 157.0 -> 158.3 mm
- net HT_VCC: track 17.7 -> 18.9 mm

Commit message: update
Parts:
- added C1, C2: CAP-US1206FAB, fab:C1206FAB
Connections:
- removed net N$27: U$2.7
- net GND1: now also C1.2, C2.2, U$2.7
- net VCC_12V: now also C1.1, C2.1
Routing:
- net GND1: track 158.3 -> 185.8 mm
- net VCC_5V: track 72.4 -> 88.9 mm, vias 3 -> 2
- net VCC_12V: track 96.3 -> 112.2 mm, vias 6 -> 4
