File: V.raspberryPi/Ecotron/EAGLE/PCB/board_0.1v.brd (EAGLE design)
At the start: 100 x 80 mm, 15 parts, among them J4 4P-2.0, J5 4P-2.0, J6 4P-2.0, U1 ADS1015, U4 PCA9546APW,112

Commit message: update
Parts:
- moved U2 14.2 mm to (22.0, 39.0)
- moved U3 14.1 mm to (22.0, 26.9)
- moved U4 13.9 mm to (34.1, 38.8), turned to 270 degrees
Routing:
- net GND: track 0.00 -> 17.5 mm, vias 0 -> 1
Changed lines of the file:
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@@
 <attribute name="PROD_ID" value="IC-12270" x="8" y="18.9" size="1.778" layer="27" rot="R270" display="off"/>
 </element>
-<element name="U2" library="adafruit" package="TSSOP20" value="" x="7.9" y="40.5"/>
-<element name="U3" library="adafruit" package="TSSOP20" value="" x="8.1" y="29.2"/>
+<element name="U2" library="adafruit" package="TSSOP20" value="" x="22" y="39"/>
+<element name="U3" library="adafruit" package="TSSOP20" value="" x="22" y="26.9"/>
 <element name="T1" library="fab_2" package="TO252" value="" x="88.6" y="15.3"/>
 <element name="T2" library="fab_2" package="TO252" value="" x="77" y="15.1"/>
@@
 <element name="J5" library="Seeed-OPL-Connector" package="HW4-2.0" value="4P-2.0" x="23.5" y="5.7"/>
 <element name="J6" library="Seeed-OPL-Connector" package="HW4-2.0" value="4P-2.0" x="36.5" y="5.7"/>
-<element name="U4" library="NXP_By_element14_Batch_1" package="SOP65P640X110-16N" value="PCA9546APW,112" x="24.7" y="28.5" rot="R90">
-<attribute name="OC_NEWARK" value="70R6610" x="24.7" y="28.5" size="1.778" layer="27" rot="R90" display="off"/>
-<attribute name="SUPPLIER" value="NXP" x="24.7" y="28.5" size="1.778" layer="27" rot="R90" display="off"/>
-<attribute name="OC_FARNELL" value="1831208" x="24.7" y="28.5" size="1.778" layer="27" rot="R90" display="off"/>
-<attribute name="MPN" value="PCA9546APW,112" x="24.7" y="28.5" size="1.778" layer="27" rot="R90" display="off"/>
-<attribute name="PACKAGE" value="TSSOP-16" x="24.7" y="28.5" size="1.778" layer="27" rot="R90" display="off"/>
+<element name="U4" library="NXP_By_element14_Batch_1" package="SOP65P640X110-16N" value="PCA9546APW,112" x="34.1" y="38.8" rot="R270">
+<attribute name="OC_NEWARK" value="70R6610" x="34.1" y="38.8" size="1.778" layer="27" rot="R270" display="off"/>
+<attribute name="SUPPLIER" value="NXP" x="34.1" y="38.8" size="1.778" layer="27" rot="R270" display="off"/>
+<attribute name="OC_FARNELL" value="1831208" x="34.1" y="38.8" size="1.778" layer="27" rot="R270" display="off"/>
+<attribute name="MPN" value="PCA9546APW,112" x="34.1" y="38.8" size="1.778" layer="27" rot="R270" display="off"/>
+<attribute name="PACKAGE" value="TSSOP-16" x="34.1" y="38.8" size="1.778" layer="27" rot="R270" display="off"/>
 </element>
 </elements>
@@
 <contactref element="J5" pad="4"/>
 <contactref element="J4" pad="4"/>
-<wire x1="10.825" y1="43.4178" x2="31.15" y2="54.57" width="0" layer="19" extent="1-1"/>
-<wire x1="11.025" y1="32.1178" x2="10.825" y2="43.4178" width="0" layer="19" extent="1-1"/>
-<wire x1="5.95" y1="18.9" x2="11.025" y2="32.1178" width="0" layer="19" extent="1-1"/>
 <wire x1="13" y1="5.7" x2="5.95" y2="18.9" width="0" layer="19" extent="1-1"/>
 <wire x1="26.5" y1="5.7" x2="13" y2="5.7" width="0" layer="19" extent="1-1"/>
 <wire x1="39.5" y1="5.7" x2="26.5" y2="5.7" width="0" layer="19" extent="1-1"/>
-<wire x1="26.986" y1="25.579" x2="11.025" y2="32.1178" width="0" layer="19" extent="1-1"/>
+<wire x1="31.814" y1="41.721" x2="24.925" y2="29.8178" width="0" layer="19" extent="1-1"/>
+<wire x1="5.95" y1="18.9" x2="24.925" y2="29.8178" width="0" layer="19" extent="1-1"/>
+<wire x1="24.925" y1="29.8178" x2="24.925" y2="41.9178" width="0" layer="19" extent="1-1"/>
+<wire x1="31.15" y1="54.57" x2="31.15" y2="48.25" width="0.4064" layer="16"/>
+<wire x1="31.15" y1="48.25" x2="30.1" y2="47.2" width="0.4064" layer="16"/>
+<wire x1="30.1" y1="47.2" x2="26.2" y2="47.2" width="0.4064" layer="16"/>
+<wire x1="26.2" y1="47.2" x2="24.9" y2="45.9" width="0.4064" layer="1"/>
+<wire x1="24.9" y1="45.9" x2="24.9" y2="41.9428" width="0.4064" layer="1"/>
+<wire x1="24.9" y1="41.9428" x2="24.925" y2="41.9178" width="0.4064" layer="1"/>
+<via x="26.2" y="47.2" extent="1-16" drill="0.6" shape="octagon"/>
 </signal>
 <signal name="GPIO17">
