File: V.raspberryPi/Ecotron/EAGLE/PCB/board_0.1v.brd (EAGLE design)
At the start: 100 x 80 mm, 15 parts, among them J4 4P-2.0, J5 4P-2.0, J6 4P-2.0, U1 ADS1015, U4 PCA9546APW,112

Commit message: nueva version Pi
Connections:
- net N$12 renamed GPIO22
- net N$14 renamed GPIO10
- net N$26 renamed GPIO8
- net N$27 renamed GPIO9
- net N$28 renamed GPIO11
- net N$31 renamed GPIO5
- net N$32 renamed GPIO6
- net N$33 renamed GPIO13
- net N$34 renamed GPIO19
- net N$35 renamed GPIO26
- net N$37 renamed GPIO7
- net N$40 renamed GPIO12
- net N$42 renamed GPIO16
- net N$43 renamed GPIO20
- net N$44 renamed GPIO21
Changed lines of the file:
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@@
 <contactref element="JP1" pad="13"/>
 </signal>
-<signal name="N$12">
+<signal name="GPIO22">
 <contactref element="JP1" pad="15"/>
 </signal>
@@
 <contactref element="JP1" pad="17"/>
 </signal>
-<signal name="N$14">
+<signal name="GPIO10">
 <contactref element="JP1" pad="19"/>
 </signal>
@@
 <contactref element="JP1" pad="22"/>
 </signal>
-<signal name="N$26">
+<signal name="GPIO8">
 <contactref element="JP1" pad="24"/>
 </signal>
-<signal name="N$27">
+<signal name="GPIO9">
 <contactref element="JP1" pad="21"/>
 </signal>
-<signal name="N$28">
+<signal name="GPIO11">
 <contactref element="JP1" pad="23"/>
 </signal>
@@
 <contactref element="JP1" pad="27"/>
 </signal>
-<signal name="N$31">
+<signal name="GPIO5">
 <contactref element="JP1" pad="29"/>
 </signal>
-<signal name="N$32">
+<signal name="GPIO6">
 <contactref element="JP1" pad="31"/>
 </signal>
-<signal name="N$33">
+<signal name="GPIO13">
 <contactref element="JP1" pad="33"/>
 </signal>
-<signal name="N$34">
+<signal name="GPIO19">
 <contactref element="JP1" pad="35"/>
 </signal>
-<signal name="N$35">
+<signal name="GPIO26">
 <contactref element="JP1" pad="37"/>
 </signal>
@@
 <contactref element="JP1" pad="39"/>
 </signal>
-<signal name="N$37">
+<signal name="GPIO7">
 <contactref element="JP1" pad="26"/>
 </signal>
@@
 <contactref element="JP1" pad="30"/>
 </signal>
-<signal name="N$40">
+<signal name="GPIO12">
 <contactref element="JP1" pad="32"/>
 </signal>
@@
 <contactref element="JP1" pad="34"/>
 </signal>
-<signal name="N$42">
+<signal name="GPIO16">
 <contactref element="JP1" pad="36"/>
 </signal>
-<signal name="N$43">
+<signal name="GPIO20">
 <contactref element="JP1" pad="38"/>
 </signal>
-<signal name="N$44">
+<signal name="GPIO21">
 <contactref element="JP1" pad="40"/>
 </signal>

Commit message: update
Connections:
- new net N$10: U3.5
- new net N$11: U3.4
- new net N$12: U3.3
- new net N$13: U3.1
- new net N$14: U3.10
- new net N$15: U3.12
- new net N$16: U3.13
- new net N$17: U3.14
- new net N$18: U3.15
- new net N$19: U3.16
- new net N$20: U3.17
- new net N$21: U3.18
- new net N$22: U3.20
- new net N$26: U3.19
- new net N$27: U3.2
- new net N$6: U3.9
- new net N$7: U3.8
- new net N$8: U3.7
- new net N$9: U3.6
- net GND: now also J4.4, J5.4, J6.4, U1.3, U2.11, U3.11, U4.8
Changed lines of the file:
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@@
 <signal name="GND">
 <contactref element="JP1" pad="6"/>
+<contactref element="U3" pad="11"/>
+<contactref element="U1" pad="3"/>
+<contactref element="U2" pad="11"/>
+<contactref element="U4" pad="8"/>
+<contactref element="J6" pad="4"/>
+<contactref element="J5" pad="4"/>
+<contactref element="J4" pad="4"/>
+<wire x1="10.825" y1="43.4178" x2="31.15" y2="54.57" width="0" layer="19" extent="1-1"/>
+<wire x1="11.025" y1="32.1178" x2="10.825" y2="43.4178" width="0" layer="19" extent="1-1"/>
+<wire x1="5.95" y1="18.9" x2="11.025" y2="32.1178" width="0" layer="19" extent="1-1"/>
+<wire x1="13" y1="5.7" x2="5.95" y2="18.9" width="0" layer="19" extent="1-1"/>
+<wire x1="26.5" y1="5.7" x2="13" y2="5.7" width="0" layer="19" extent="1-1"/>
+<wire x1="39.5" y1="5.7" x2="26.5" y2="5.7" width="0" layer="19" extent="1-1"/>
+<wire x1="26.986" y1="25.579" x2="11.025" y2="32.1178" width="0" layer="19" extent="1-1"/>
 </signal>
 <signal name="GPIO17">
@@
 <contactref element="U4" pad="16"/>
 </signal>
+<signal name="N$6">
+<contactref element="U3" pad="9"/>
+</signal>
+<signal name="N$7">
+<contactref element="U3" pad="8"/>
+</signal>
+<signal name="N$8">
+<contactref element="U3" pad="7"/>
+</signal>
+<signal name="N$9">
+<contactref element="U3" pad="6"/>
+</signal>
+<signal name="N$10">
+<contactref element="U3" pad="5"/>
+</signal>
+<signal name="N$11">
+<contactref element="U3" pad="4"/>
+</signal>
+<signal name="N$12">
+<contactref element="U3" pad="3"/>
+</signal>
+<signal name="N$13">
+<contactref element="U3" pad="1"/>
+</signal>
+<signal name="N$14">
+<contactref element="U3" pad="10"/>
+</signal>
+<signal name="N$15">
+<contactref element="U3" pad="12"/>
+</signal>
+<signal name="N$16">
+<contactref element="U3" pad="13"/>
+</signal>
+<signal name="N$17">
+<contactref element="U3" pad="14"/>
+</signal>
+<signal name="N$18">
+<contactref element="U3" pad="15"/>
+</signal>
+<signal name="N$19">
+<contactref element="U3" pad="16"/>
+</signal>
+<signal name="N$20">
+<contactref element="U3" pad="17"/>
+</signal>
+<signal name="N$21">
+<contactref element="U3" pad="18"/>
+</signal>
+<signal name="N$22">
+<contactref element="U3" pad="20"/>
+</signal>
+<signal name="N$26">
+<contactref element="U3" pad="19"/>
+</signal>
+<signal name="N$27">
+<contactref element="U3" pad="2"/>
+</signal>
 </signals>

Commit message: u
Parts:
- removed U2: (no value), adafruit:TSSOP20
- added C1, C2: CAP-US1206FAB, fab:C1206FAB
Connections:
- net GND: now also C1.2, C2.2; no longer U2.11
- net N$26: now also C1.1
- net N$27: now also C2.1
Changed lines of the file:
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@@
 <attribute name="PROD_ID" value="IC-12270" x="8" y="18.9" size="1.778" layer="27" rot="R270" display="off"/>
 </element>
-<element name="U2" library="adafruit" package="TSSOP20" value="" x="7.9" y="40.5"/>
 <element name="U3" library="adafruit" package="TSSOP20" value="" x="8.1" y="29.2"/>
 <element name="T1" library="fab_2" package="TO252" value="" x="88.6" y="15.3"/>
@@
 <attribute name="PACKAGE" value="TSSOP-16" x="24.7" y="28.5" size="1.778" layer="27" rot="R90" display="off"/>
 </element>
+<element name="C1" library="fab" package="C1206FAB" value="CAP-US1206FAB" x="2.4" y="-4.1"/>
+<element name="C2" library="fab" package="C1206FAB" value="CAP-US1206FAB" x="2.4" y="-10.5"/>
 </elements>
 <signals>
@@
 <contactref element="U3" pad="11"/>
 <contactref element="U1" pad="3"/>
-<contactref element="U2" pad="11"/>
 <contactref element="U4" pad="8"/>
 <contactref element="J6" pad="4"/>
 <contactref element="J5" pad="4"/>
 <contactref element="J4" pad="4"/>
-<wire x1="10.825" y1="43.4178" x2="31.15" y2="54.57" width="0" layer="19" extent="1-1"/>
-<wire x1="11.025" y1="32.1178" x2="10.825" y2="43.4178" width="0" layer="19" extent="1-1"/>
+<contactref element="C1" pad="2"/>
+<contactref element="C2" pad="2"/>
+<wire x1="26.986" y1="25.579" x2="31.15" y2="54.57" width="0" layer="19" extent="1-1"/>
+<wire x1="11.025" y1="32.1178" x2="26.986" y2="25.579" width="0" layer="19" extent="1-1"/>
 <wire x1="5.95" y1="18.9" x2="11.025" y2="32.1178" width="0" layer="19" extent="1-1"/>
 <wire x1="13" y1="5.7" x2="5.95" y2="18.9" width="0" layer="19" extent="1-1"/>
+<wire x1="4.051" y1="-4.1" x2="13" y2="5.7" width="0" layer="19" extent="1-1"/>
+<wire x1="4.051" y1="-10.5" x2="4.051" y2="-4.1" width="0" layer="19" extent="1-1"/>
 <wire x1="26.5" y1="5.7" x2="13" y2="5.7" width="0" layer="19" extent="1-1"/>
 <wire x1="39.5" y1="5.7" x2="26.5" y2="5.7" width="0" layer="19" extent="1-1"/>
-<wire x1="26.986" y1="25.579" x2="11.025" y2="32.1178" width="0" layer="19" extent="1-1"/>
 </signal>
 <signal name="GPIO17">
@@
 <signal name="N$26">
 <contactref element="U3" pad="19"/>
+<contactref element="C1" pad="1"/>
+<wire x1="0.749" y1="-4.1" x2="5.825" y2="32.1178" width="0" layer="19" extent="1-1"/>
 </signal>
 <signal name="N$27">
 <contactref element="U3" pad="2"/>
+<contactref element="C2" pad="1"/>
+<wire x1="0.749" y1="-10.5" x2="5.825" y2="26.2822" width="0" layer="19" extent="1-1"/>
 </signal>
 </signals>

Commit message: seedstudio finish
Parts:
- removed C1, C2: CAP-US1206FAB, fab:C1206FAB
- added U2: (no value), adafruit:TSSOP20
- moved U3 14.1 mm to (22.0, 26.9)
- moved U4 13.9 mm to (34.1, 38.8), turned to 270 degrees
Connections:
- net GND: now also U2.11; no longer C1.2, C2.2
- net N$26: no longer C1.1
- net N$27: no longer C2.1
Routing:
- net GND: track 0.00 -> 134.5 mm, vias 0 -> 1
Changed lines of the file:
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@@
 <attribute name="PROD_ID" value="IC-12270" x="8" y="18.9" size="1.778" layer="27" rot="R270" display="off"/>
 </element>
-<element name="U3" library="adafruit" package="TSSOP20" value="" x="8.1" y="29.2"/>
+<element name="U2" library="adafruit" package="TSSOP20" value="" x="22" y="39"/>
+<element name="U3" library="adafruit" package="TSSOP20" value="" x="22" y="26.9"/>
 <element name="T1" library="fab_2" package="TO252" value="" x="88.6" y="15.3"/>
 <element name="T2" library="fab_2" package="TO252" value="" x="77" y="15.1"/>
@@
 <element name="J5" library="Seeed-OPL-Connector" package="HW4-2.0" value="4P-2.0" x="23.5" y="5.7"/>
 <element name="J6" library="Seeed-OPL-Connector" package="HW4-2.0" value="4P-2.0" x="36.5" y="5.7"/>
-<element name="U4" library="NXP_By_element14_Batch_1" package="SOP65P640X110-16N" value="PCA9546APW,112" x="24.7" y="28.5" rot="R90">
-<attribute name="OC_NEWARK" value="70R6610" x="24.7" y="28.5" size="1.778" layer="27" rot="R90" display="off"/>
-<attribute name="SUPPLIER" value="NXP" x="24.7" y="28.5" size="1.778" layer="27" rot="R90" display="off"/>
-<attribute name="OC_FARNELL" value="1831208" x="24.7" y="28.5" size="1.778" layer="27" rot="R90" display="off"/>
-<attribute name="MPN" value="PCA9546APW,112" x="24.7" y="28.5" size="1.778" layer="27" rot="R90" display="off"/>
-<attribute name="PACKAGE" value="TSSOP-16" x="24.7" y="28.5" size="1.778" layer="27" rot="R90" display="off"/>
+<element name="U4" library="NXP_By_element14_Batch_1" package="SOP65P640X110-16N" value="PCA9546APW,112" x="34.1" y="38.8" rot="R270">
+<attribute name="OC_NEWARK" value="70R6610" x="34.1" y="38.8" size="1.778" layer="27" rot="R270" display="off"/>
+<attribute name="SUPPLIER" value="NXP" x="34.1" y="38.8" size="1.778" layer="27" rot="R270" display="off"/>
+<attribute name="OC_FARNELL" value="1831208" x="34.1" y="38.8" size="1.778" layer="27" rot="R270" display="off"/>
+<attribute name="MPN" value="PCA9546APW,112" x="34.1" y="38.8" size="1.778" layer="27" rot="R270" display="off"/>
+<attribute name="PACKAGE" value="TSSOP-16" x="34.1" y="38.8" size="1.778" layer="27" rot="R270" display="off"/>
 </element>
-<element name="C1" library="fab" package="C1206FAB" value="CAP-US1206FAB" x="2.4" y="-4.1"/>
-<element name="C2" library="fab" package="C1206FAB" value="CAP-US1206FAB" x="2.4" y="-10.5"/>
 </elements>
 <signals>
@@
 <contactref element="U3" pad="11"/>
 <contactref element="U1" pad="3"/>
+<contactref element="U2" pad="11"/>
 <contactref element="U4" pad="8"/>
 <contactref element="J6" pad="4"/>
 <contactref element="J5" pad="4"/>
 <contactref element="J4" pad="4"/>
-<contactref element="C1" pad="2"/>
-<contactref element="C2" pad="2"/>
-<wire x1="26.986" y1="25.579" x2="31.15" y2="54.57" width="0" layer="19" extent="1-1"/>
-<wire x1="11.025" y1="32.1178" x2="26.986" y2="25.579" width="0" layer="19" extent="1-1"/>
-<wire x1="5.95" y1="18.9" x2="11.025" y2="32.1178" width="0" layer="19" extent="1-1"/>
-<wire x1="13" y1="5.7" x2="5.95" y2="18.9" width="0" layer="19" extent="1-1"/>
-<wire x1="4.051" y1="-4.1" x2="13" y2="5.7" width="0" layer="19" extent="1-1"/>
-<wire x1="4.051" y1="-10.5" x2="4.051" y2="-4.1" width="0" layer="19" extent="1-1"/>
-<wire x1="26.5" y1="5.7" x2="13" y2="5.7" width="0" layer="19" extent="1-1"/>
-<wire x1="39.5" y1="5.7" x2="26.5" y2="5.7" width="0" layer="19" extent="1-1"/>
+<wire x1="31.15" y1="54.57" x2="31.15" y2="48.25" width="0.4064" layer="16"/>
+<wire x1="31.15" y1="48.25" x2="30.1" y2="47.2" width="0.4064" layer="16"/>
+<wire x1="30.1" y1="47.2" x2="26.2" y2="47.2" width="0.4064" layer="16"/>
+<wire x1="26.2" y1="47.2" x2="24.9" y2="45.9" width="0.4064" layer="1"/>
+<wire x1="24.9" y1="45.9" x2="24.9" y2="41.9428" width="0.4064" layer="1"/>
+<wire x1="24.9" y1="41.9428" x2="24.925" y2="41.9178" width="0.4064" layer="1"/>
+<via x="26.2" y="47.2" extent="1-16" drill="0.6" shape="octagon"/>
+<wire x1="24.925" y1="41.9178" x2="27.8" y2="41.9178" width="0.4064" layer="1"/>
+<wire x1="27.8" y1="41.9178" x2="31.814" y2="41.9178" width="0.4064" layer="1"/>
+<wire x1="31.814" y1="41.9178" x2="31.814" y2="41.721" width="0.4064" layer="1"/>
+<wire x1="24.925" y1="29.8178" x2="26.2178" y2="29.8178" width="0.4064" layer="1"/>
+<wire x1="26.2178" y1="29.8178" x2="27.5" y2="31.1" width="0.4064" layer="1"/>
+<wire x1="27.5" y1="31.1" x2="27.5" y2="31.6" width="0.4064" layer="1"/>
+<wire x1="27.5" y1="31.6" x2="27.5" y2="41.6178" width="0.4064" layer="1"/>
+<wire x1="27.5" y1="41.6178" x2="27.8" y2="41.9178" width="0.4064" layer="1"/>
+<wire x1="5.95" y1="18.9" x2="4.9" y2="18.9" width="0.4064" layer="1"/>
+<wire x1="4.9" y1="18.9" x2="3.95" y2="19.85" width="0.4064" layer="1"/>
+<wire x1="3.95" y1="19.85" x2="3.9" y2="19.9" width="0.4064" layer="1"/>
+<wire x1="3.9" y1="19.9" x2="3.9" y2="29.4" width="0.4064" layer="1"/>
+<wire x1="3.9" y1="29.4" x2="7.5" y2="33" width="0.4064" layer="1"/>
+<wire x1="7.5" y1="33" x2="26.1" y2="33" width="0.4064" layer="1"/>
+<wire x1="26.1" y1="33" x2="27.5" y2="31.6" width="0.4064" layer="1"/>
+<wire x1="13" y1="5.7" x2="13" y2="8.9" width="0.4064" layer="1"/>
+<wire x1="13" y1="8.9" x2="14.7" y2="10.6" width="0.4064" layer="1"/>
+<wire x1="14.7" y1="10.6" x2="27.7" y2="10.6" width="0.4064" layer="1"/>
+<wire x1="27.7" y1="10.6" x2="38" y2="10.6" width="0.4064" layer="1"/>
+<wire x1="38" y1="10.6" x2="39.5" y2="9.1" width="0.4064" layer="1"/>
+<wire x1="39.5" y1="9.1" x2="39.5" y2="5.7" width="0.4064" layer="1"/>
+<wire x1="26.5" y1="5.7" x2="26.5" y2="9.4" width="0.4064" layer="1"/>
+<wire x1="26.5" y1="9.4" x2="27.7" y2="10.6" width="0.4064" layer="1"/>
+<wire x1="14.7" y1="10.6" x2="14.6" y2="10.6" width="0.4064" layer="1"/>
+<wire x1="14.6" y1="10.6" x2="12.5" y2="12.7" width="0.4064" layer="1"/>
+<wire x1="12.5" y1="12.7" x2="4.8" y2="12.7" width="0.4064" layer="1"/>
+<wire x1="4.8" y1="12.7" x2="3.8" y2="13.7" width="0.4064" layer="1"/>
+<wire x1="3.8" y1="13.7" x2="3.8" y2="19.7" width="0.4064" layer="1"/>
+<wire x1="3.8" y1="19.7" x2="3.95" y2="19.85" width="0.4064" layer="1"/>
 </signal>
 <signal name="GPIO17">
@@
 <signal name="N$26">
 <contactref element="U3" pad="19"/>
-<contactref element="C1" pad="1"/>
-<wire x1="0.749" y1="-4.1" x2="5.825" y2="32.1178" width="0" layer="19" extent="1-1"/>
 </signal>
 <signal name="N$27">
 <contactref element="U3" pad="2"/>
-<contactref element="C2" pad="1"/>
-<wire x1="0.749" y1="-10.5" x2="5.825" y2="26.2822" width="0" layer="19" extent="1-1"/>
 </signal>
 </signals>
