File: V.raspberryPi/Ecotron/EAGLE/PCB/board_0.1v.sch (EAGLE design)
At the start: 15 parts, among them J4 4P-2.0, J5 4P-2.0, J6 4P-2.0, U1 ADS1015, U4 PCA9546APW,112

Commit message: nueva version Pi
Connections:
- net N$12 renamed GPIO22
- net N$14 renamed GPIO10
- net N$26 renamed GPIO8
- net N$27 renamed GPIO9
- net N$28 renamed GPIO11
- net N$31 renamed GPIO5
- net N$32 renamed GPIO6
- net N$33 renamed GPIO13
- net N$34 renamed GPIO19
- net N$35 renamed GPIO26
- net N$37 renamed GPIO7
- net N$40 renamed GPIO12
- net N$42 renamed GPIO16
- net N$43 renamed GPIO20
- net N$44 renamed GPIO21
Changed lines of the file:
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@@
 </segment>
 </net>
-<net name="N$12" class="0">
+<net name="GPIO22" class="0">
 <segment>
 <pinref part="JP1" gate="A" pin="15"/>
 <wire x1="165.1" y1="121.92" x2="172.72" y2="121.92" width="0.1524" layer="91"/>
+<label x="175.26" y="121.92" size="1.27" layer="95" xref="yes"/>
 </segment>
 </net>
@@
 </segment>
 </net>
-<net name="N$14" class="0">
+<net name="GPIO10" class="0">
 <segment>
 <pinref part="JP1" gate="A" pin="19"/>
 <wire x1="165.1" y1="127" x2="172.72" y2="127" width="0.1524" layer="91"/>
+<label x="175.26" y="127" size="1.27" layer="95" xref="yes"/>
 </segment>
 </net>
@@
 <pinref part="JP1" gate="A" pin="18"/>
 <wire x1="157.48" y1="124.46" x2="149.86" y2="124.46" width="0.1524" layer="91"/>
+<label x="147.32" y="124.46" size="1.27" layer="95" rot="R180" xref="yes"/>
 </segment>
 </net>
@@
 <pinref part="JP1" gate="A" pin="22"/>
 <wire x1="157.48" y1="129.54" x2="149.86" y2="129.54" width="0.1524" layer="91"/>
-</segment>
-</net>
-<net name="N$26" class="0">
+<label x="147.32" y="129.54" size="1.27" layer="95" rot="R180" xref="yes"/>
+</segment>
+</net>
+<net name="GPIO8" class="0">
 <segment>
 <pinref part="JP1" gate="A" pin="24"/>
 <wire x1="157.48" y1="132.08" x2="149.86" y2="132.08" width="0.1524" layer="91"/>
-</segment>
-</net>
-<net name="N$27" class="0">
+<label x="147.32" y="132.08" size="1.27" layer="95" rot="R180" xref="yes"/>
+</segment>
+</net>
+<net name="GPIO9" class="0">
 <segment>
 <pinref part="JP1" gate="A" pin="21"/>
 <wire x1="165.1" y1="129.54" x2="172.72" y2="129.54" width="0.1524" layer="91"/>
-</segment>
-</net>
-<net name="N$28" class="0">
+<label x="175.26" y="129.54" size="1.27" layer="95" xref="yes"/>
+</segment>
+</net>
+<net name="GPIO11" class="0">
 <segment>
 <pinref part="JP1" gate="A" pin="23"/>
 <wire x1="165.1" y1="132.08" x2="172.72" y2="132.08" width="0.1524" layer="91"/>
+<label x="175.26" y="132.08" size="1.27" layer="95" xref="yes"/>
 </segment>
 </net>
@@
 <pinref part="JP1" gate="A" pin="27"/>
 <wire x1="165.1" y1="137.16" x2="172.72" y2="137.16" width="0.1524" layer="91"/>
-</segment>
-</net>
-<net name="N$31" class="0">
+<label x="175.26" y="137.16" size="1.27" layer="95" xref="yes"/>
+</segment>
+</net>
+<net name="GPIO5" class="0">
 <segment>
 <pinref part="JP1" gate="A" pin="29"/>
 <wire x1="165.1" y1="139.7" x2="172.72" y2="139.7" width="0.1524" layer="91"/>
-</segment>
-</net>
-<net name="N$32" class="0">
+<label x="175.26" y="139.7" size="1.27" layer="95" xref="yes"/>
+</segment>
+</net>
+<net name="GPIO6" class="0">
 <segment>
 <pinref part="JP1" gate="A" pin="31"/>
 <wire x1="165.1" y1="142.24" x2="172.72" y2="142.24" width="0.1524" layer="91"/>
-</segment>
-</net>
-<net name="N$33" class="0">
+<label x="175.26" y="142.24" size="1.27" layer="95" xref="yes"/>
+</segment>
+</net>
+<net name="GPIO13" class="0">
 <segment>
 <pinref part="JP1" gate="A" pin="33"/>
 <wire x1="165.1" y1="144.78" x2="172.72" y2="144.78" width="0.1524" layer="91"/>
-</segment>
-</net>
-<net name="N$34" class="0">
+<label x="175.26" y="144.78" size="1.27" layer="95" xref="yes"/>
+</segment>
+</net>
+<net name="GPIO19" class="0">
 <segment>
 <pinref part="JP1" gate="A" pin="35"/>
 <wire x1="165.1" y1="147.32" x2="172.72" y2="147.32" width="0.1524" layer="91"/>
-</segment>
-</net>
-<net name="N$35" class="0">
+<label x="175.26" y="147.32" size="1.27" layer="95" xref="yes"/>
+</segment>
+</net>
+<net name="GPIO26" class="0">
 <segment>
 <pinref part="JP1" gate="A" pin="37"/>
 <wire x1="165.1" y1="149.86" x2="172.72" y2="149.86" width="0.1524" layer="91"/>
+<label x="175.26" y="149.86" size="1.27" layer="95" xref="yes"/>
 </segment>
 </net>
@@
 </segment>
 </net>
-<net name="N$37" class="0">
+<net name="GPIO7" class="0">
 <segment>
 <pinref part="JP1" gate="A" pin="26"/>
 <wire x1="157.48" y1="134.62" x2="149.86" y2="134.62" width="0.1524" layer="91"/>
+<label x="147.32" y="134.62" size="1.27" layer="95" rot="R180" xref="yes"/>
 </segment>
 </net>
@@
 <pinref part="JP1" gate="A" pin="28"/>
 <wire x1="157.48" y1="137.16" x2="149.86" y2="137.16" width="0.1524" layer="91"/>
+<label x="147.32" y="137.16" size="1.27" layer="95" rot="R180" xref="yes"/>
 </segment>
 </net>
@@
 </segment>
 </net>
-<net name="N$40" class="0">
+<net name="GPIO12" class="0">
 <segment>
 <pinref part="JP1" gate="A" pin="32"/>
 <wire x1="157.48" y1="142.24" x2="149.86" y2="142.24" width="0.1524" layer="91"/>
+<label x="147.32" y="142.24" size="1.27" layer="95" rot="R180" xref="yes"/>
 </segment>
 </net>
@@
 </segment>
 </net>
-<net name="N$42" class="0">
+<net name="GPIO16" class="0">
 <segment>
 <pinref part="JP1" gate="A" pin="36"/>
 <wire x1="157.48" y1="147.32" x2="149.86" y2="147.32" width="0.1524" layer="91"/>
-</segment>
-</net>
-<net name="N$43" class="0">
+<label x="147.32" y="147.32" size="1.27" layer="95" rot="R180" xref="yes"/>
+</segment>
+</net>
+<net name="GPIO20" class="0">
 <segment>
 <pinref part="JP1" gate="A" pin="38"/>
 <wire x1="157.48" y1="149.86" x2="149.86" y2="149.86" width="0.1524" layer="91"/>
-</segment>
-</net>
-<net name="N$44" class="0">
+<label x="147.32" y="149.86" size="1.27" layer="95" rot="R180" xref="yes"/>
+</segment>
+</net>
+<net name="GPIO21" class="0">
 <segment>
 <pinref part="JP1" gate="A" pin="40"/>
 <wire x1="157.48" y1="152.4" x2="149.86" y2="152.4" width="0.1524" layer="91"/>
+<label x="147.32" y="152.4" size="1.27" layer="95" rot="R180" xref="yes"/>
 </segment>
 </net>
@@
 <pinref part="JP1" gate="A" pin="4"/>
 <wire x1="157.48" y1="106.68" x2="149.86" y2="106.68" width="0.1524" layer="91"/>
-</segment>
-</net>
+<label x="147.32" y="106.68" size="1.27" layer="95" rot="R180" xref="yes"/>
+</segment>
+</net>

Commit message: update
Connections:
- new net N$10: U3.A4
- new net N$11: U3.A3
- new net N$12: U3.A2
- new net N$13: U3.A1
- new net N$14: U3.OE
- new net N$15: U3.B8
- new net N$16: U3.B7
- new net N$17: U3.B6
- new net N$18: U3.B5
- new net N$19: U3.B4
- new net N$20: U3.B3
- new net N$21: U3.B2
- new net N$22: U3.B1
- new net N$26: U3.VCCB
- new net N$27: U3.VCCA
- new net N$6: U3.A8
- new net N$7: U3.A7
- new net N$8: U3.A6
- new net N$9: U3.A5
- net GND: now also J4.4, J5.4, J6.4, U1.VSS, U2.GND, U3.GND, U4.VSS
Other:
- moved on the sheet: J4, J5, J6
Changed lines of the file:
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@@
 <setting verticaltext="up"/>
 </settings>
-<grid distance="0.1" unitdist="inch" unit="inch" style="lines" multiple="1" display="no" altdistance="0.01" altunitdist="inch" altunit="inch"/>
+<grid distance="0.1" unitdist="inch" unit="inch" style="lines" multiple="1" display="yes" altdistance="0.01" altunitdist="inch" altunit="inch"/>
 <layers>
 <layer number="1" name="Top" color="4" fill="1" visible="no" active="no"/>
@@
 <part name="J6" library="Seeed-OPL-Connector" deviceset="GROVE-CONNECTOR-DIP(4P-2.0)" device="" value="4P-2.0"/>
 <part name="U4" library="NXP_By_element14_Batch_1" deviceset="PCA9546APW,112" device=""/>
+<part name="SUPPLY1" library="supply2" deviceset="GND" device=""/>
+<part name="SUPPLY2" library="supply2" deviceset="GND" device=""/>
+<part name="SUPPLY3" library="supply2" deviceset="GND" device=""/>
+<part name="SUPPLY4" library="supply2" deviceset="GND" device=""/>
+<part name="SUPPLY5" library="supply2" deviceset="GND" device=""/>
+<part name="SUPPLY6" library="supply2" deviceset="GND" device=""/>
+<part name="SUPPLY7" library="supply2" deviceset="GND" device=""/>
 </parts>
 <sheets>
@@
 <instance part="T5" gate="A" x="40.64" y="17.78"/>
 <instance part="T6" gate="A" x="38.1" y="2.54"/>
-<instance part="J4" gate="G$1" x="185.42" y="68.58"/>
-<instance part="J5" gate="G$1" x="167.64" y="68.58"/>
-<instance part="J6" gate="G$1" x="147.32" y="71.12"/>
+<instance part="J4" gate="G$1" x="191.77" y="69.85"/>
+<instance part="J5" gate="G$1" x="168.91" y="69.85"/>
+<instance part="J6" gate="G$1" x="148.59" y="69.85"/>
 <instance part="U4" gate="A" x="116.84" y="53.34"/>
+<instance part="SUPPLY1" gate="GND" x="106.68" y="154.94"/>
+<instance part="SUPPLY2" gate="GND" x="45.72" y="45.72"/>
+<instance part="SUPPLY3" gate="GND" x="43.18" y="154.94"/>
+<instance part="SUPPLY4" gate="GND" x="91.44" y="17.78"/>
+<instance part="SUPPLY5" gate="GND" x="139.7" y="58.42"/>
+<instance part="SUPPLY6" gate="GND" x="160.02" y="58.42"/>
+<instance part="SUPPLY7" gate="GND" x="182.88" y="58.42"/>
 </instances>
 <busses>
@@
 <label x="147.32" y="109.22" size="1.016" layer="95" rot="R180" xref="yes"/>
 </segment>
+<segment>
+<pinref part="U3" gate="G$1" pin="GND"/>
+<wire x1="88.9" y1="152.4" x2="88.9" y2="157.48" width="0.1524" layer="91"/>
+<wire x1="88.9" y1="157.48" x2="106.68" y2="157.48" width="0.1524" layer="91"/>
+<pinref part="SUPPLY1" gate="GND" pin="GND"/>
+</segment>
+<segment>
+<pinref part="SUPPLY2" gate="GND" pin="GND"/>
+<pinref part="U1" gate="G$1" pin="VSS"/>
+<wire x1="45.72" y1="48.26" x2="45.72" y2="53.34" width="0.1524" layer="91"/>
+</segment>
+<segment>
+<pinref part="U2" gate="G$1" pin="GND"/>
+<wire x1="30.48" y1="152.4" x2="30.48" y2="160.02" width="0.1524" layer="91"/>
+<wire x1="30.48" y1="160.02" x2="43.18" y2="160.02" width="0.1524" layer="91"/>
+<pinref part="SUPPLY3" gate="GND" pin="GND"/>
+<wire x1="43.18" y1="160.02" x2="43.18" y2="157.48" width="0.1524" layer="91"/>
+</segment>
+<segment>
+<pinref part="SUPPLY4" gate="GND" pin="GND"/>
+<wire x1="91.44" y1="20.32" x2="91.44" y2="25.4" width="0.1524" layer="91"/>
+<pinref part="U4" gate="A" pin="VSS"/>
+<wire x1="91.44" y1="25.4" x2="99.06" y2="25.4" width="0.1524" layer="91"/>
+</segment>
+<segment>
+<pinref part="J6" gate="G$1" pin="4"/>
+<wire x1="144.78" y1="66.04" x2="139.7" y2="66.04" width="0.1524" layer="91"/>
+<wire x1="139.7" y1="66.04" x2="139.7" y2="60.96" width="0.1524" layer="91"/>
+<pinref part="SUPPLY5" gate="GND" pin="GND"/>
+</segment>
+<segment>
+<pinref part="SUPPLY6" gate="GND" pin="GND"/>
+<wire x1="160.02" y1="60.96" x2="160.02" y2="66.04" width="0.1524" layer="91"/>
+<pinref part="J5" gate="G$1" pin="4"/>
+<wire x1="160.02" y1="66.04" x2="165.1" y2="66.04" width="0.1524" layer="91"/>
+</segment>
+<segment>
+<wire x1="187.96" y1="66.04" x2="182.88" y2="66.04" width="0.1524" layer="91"/>
+<pinref part="SUPPLY7" gate="GND" pin="GND"/>
+<wire x1="182.88" y1="66.04" x2="182.88" y2="60.96" width="0.1524" layer="91"/>
+<pinref part="J4" gate="G$1" pin="4"/>
+</segment>
 </net>
 <net name="GPIO17" class="0">
@@
 </segment>
 </net>
+<net name="N$6" class="0">
+<segment>
+<pinref part="U3" gate="G$1" pin="A8"/>
+<wire x1="104.14" y1="142.24" x2="111.76" y2="142.24" width="0.1524" layer="91"/>
+<label x="114.3" y="142.24" size="1.27" layer="95" xref="yes"/>
+</segment>
+</net>
+<net name="N$7" class="0">
+<segment>
+<pinref part="U3" gate="G$1" pin="A7"/>
+<wire x1="104.14" y1="139.7" x2="111.76" y2="139.7" width="0.1524" layer="91"/>
+<label x="114.3" y="139.7" size="1.27" layer="95" xref="yes"/>
+</segment>
+</net>
+<net name="N$8" class="0">
+<segment>
+<pinref part="U3" gate="G$1" pin="A6"/>
+<wire x1="104.14" y1="137.16" x2="111.76" y2="137.16" width="0.1524" layer="91"/>
+<label x="114.3" y="137.16" size="1.27" layer="95" xref="yes"/>
+</segment>
+</net>
+<net name="N$9" class="0">
+<segment>
+<pinref part="U3" gate="G$1" pin="A5"/>
+<wire x1="104.14" y1="134.62" x2="111.76" y2="134.62" width="0.1524" layer="91"/>
+<label x="114.3" y="134.62" size="1.27" layer="95" xref="yes"/>
+</segment>
+</net>
+<net name="N$10" class="0">
+<segment>
+<pinref part="U3" gate="G$1" pin="A4"/>
+<wire x1="104.14" y1="132.08" x2="111.76" y2="132.08" width="0.1524" layer="91"/>
+<label x="114.3" y="132.08" size="1.27" layer="95" xref="yes"/>
+</segment>
+</net>
+<net name="N$11" class="0">
+<segment>
+<pinref part="U3" gate="G$1" pin="A3"/>
+<wire x1="104.14" y1="129.54" x2="111.76" y2="129.54" width="0.1524" layer="91"/>
+<label x="114.3" y="129.54" size="1.27" layer="95" xref="yes"/>
+</segment>
+</net>
+<net name="N$12" class="0">
+<segment>
+<pinref part="U3" gate="G$1" pin="A2"/>
+<wire x1="104.14" y1="127" x2="111.76" y2="127" width="0.1524" layer="91"/>
+<label x="114.3" y="127" size="1.27" layer="95" xref="yes"/>
+</segment>
+</net>
+<net name="N$13" class="0">
+<segment>
+<pinref part="U3" gate="G$1" pin="A1"/>
+<wire x1="104.14" y1="124.46" x2="111.76" y2="124.46" width="0.1524" layer="91"/>
+<label x="114.3" y="124.46" size="1.27" layer="95" xref="yes"/>
+</segment>
+</net>
+<net name="N$14" class="0">
+<segment>
+<pinref part="U3" gate="G$1" pin="OE"/>
+<wire x1="104.14" y1="116.84" x2="111.76" y2="116.84" width="0.1524" layer="91"/>
+<label x="114.3" y="116.84" size="1.27" layer="95" xref="yes"/>
+</segment>
+</net>
+<net name="N$15" class="0">
+<segment>
+<pinref part="U3" gate="G$1" pin="B8"/>
+<wire x1="73.66" y1="142.24" x2="66.04" y2="142.24" width="0.1524" layer="91"/>
+<label x="63.5" y="142.24" size="1.27" layer="95" rot="R180" xref="yes"/>
+</segment>
+</net>
+<net name="N$16" class="0">
+<segment>
+<pinref part="U3" gate="G$1" pin="B7"/>
+<wire x1="73.66" y1="139.7" x2="66.04" y2="139.7" width="0.1524" layer="91"/>
+<label x="63.5" y="139.7" size="1.27" layer="95" rot="R180" xref="yes"/>
+</segment>
+</net>
+<net name="N$17" class="0">
+<segment>
+<pinref part="U3" gate="G$1" pin="B6"/>
+<wire x1="73.66" y1="137.16" x2="66.04" y2="137.16" width="0.1524" layer="91"/>
+<label x="63.5" y="137.16" size="1.27" layer="95" rot="R180" xref="yes"/>
+</segment>
+</net>
+<net name="N$18" class="0">
+<segment>
+<pinref part="U3" gate="G$1" pin="B5"/>
+<wire x1="73.66" y1="134.62" x2="66.04" y2="134.62" width="0.1524" layer="91"/>
+<label x="63.5" y="134.62" size="1.27" layer="95" rot="R180" xref="yes"/>
+</segment>
+</net>
+<net name="N$19" class="0">
+<segment>
+<pinref part="U3" gate="G$1" pin="B4"/>
+<wire x1="73.66" y1="132.08" x2="66.04" y2="132.08" width="0.1524" layer="91"/>
+<label x="63.5" y="132.08" size="1.27" layer="95" rot="R180" xref="yes"/>
+</segment>
+</net>
+<net name="N$20" class="0">
+<segment>
+<pinref part="U3" gate="G$1" pin="B3"/>
+<wire x1="73.66" y1="129.54" x2="66.04" y2="129.54" width="0.1524" layer="91"/>
+<label x="63.5" y="129.54" size="1.27" layer="95" rot="R180" xref="yes"/>
+</segment>
+</net>
+<net name="N$21" class="0">
+<segment>
+<pinref part="U3" gate="G$1" pin="B2"/>
+<wire x1="73.66" y1="127" x2="66.04" y2="127" width="0.1524" layer="91"/>
+<label x="63.5" y="127" size="1.27" layer="95" rot="R180" xref="yes"/>
+</segment>
+</net>
+<net name="N$22" class="0">
+<segment>
+<pinref part="U3" gate="G$1" pin="B1"/>
+<wire x1="73.66" y1="124.46" x2="66.04" y2="124.46" width="0.1524" layer="91"/>
+<label x="63.5" y="124.46" size="1.27" layer="95" rot="R180" xref="yes"/>
+</segment>
+</net>
+<net name="N$26" class="0">
+<segment>
+<pinref part="U3" gate="G$1" pin="VCCB"/>
+<wire x1="86.36" y1="109.22" x2="86.36" y2="101.6" width="0.1524" layer="91"/>
+<wire x1="86.36" y1="101.6" x2="78.74" y2="101.6" width="0.1524" layer="91"/>
+<label x="76.2" y="101.6" size="1.27" layer="95" rot="R180" xref="yes"/>
+</segment>
+</net>
+<net name="N$27" class="0">
+<segment>
+<pinref part="U3" gate="G$1" pin="VCCA"/>
+<wire x1="91.44" y1="109.22" x2="91.44" y2="101.6" width="0.1524" layer="91"/>
+<wire x1="91.44" y1="101.6" x2="99.06" y2="101.6" width="0.1524" layer="91"/>
+<label x="101.6" y="101.6" size="1.27" layer="95" xref="yes"/>
+</segment>
+</net>

Commit message: u
Parts:
- removed U2: (no value), adafruit:TXB0108PWR
- added C1, C2: CAP-US1206FAB, fab:CAP-US1206FAB
Connections:
- net GND: now also C1.2, C2.2; no longer U2.GND
- net N$26: now also C1.1
- net N$27: now also C2.1
Other:
- moved on the sheet: J4, J5, J6, JP1, U$1, U1, U3
