File: V.raspberryPi/Ecotron/EAGLE/PCB/Module_T+H_01v.brd (EAGLE design)
At the start: 43.2 x 41.9 mm, 12 parts, among them J1 4P-2.0, J2 4P-2.0

Commit message: seedstudio finish
Parts:
- added E$1, E$4: (no value), Seeed-OPL-Connector:1P-100/60MIL
- added E$2: GND, Seeed-OPL-Connector:1P-100/60MIL
- added E$5: gnd, Seeed-OPL-Connector:1P-100/60MIL
Routing:
- net SDA: track 58.9 -> 53.0 mm, vias 0 -> 2
- net GND: vias 0 -> 7
- added copper zone on layer 1, net GND
- added copper zone on layer 16, net GND
Other:
- board size 43.2 x 41.9 mm -> 44.3 x 41.9 mm
- board text added: "2017"
- board text added: "nanusefue@gmail.com"
