File: V.raspberryPi/Ecotron/EAGLE/PCB/Module_T+H_01v.sch (EAGLE design)
At the start: 12 parts, among them J1 4P-2.0, J2 4P-2.0

Commit message: seedstudio finish
Parts:
- C1: value (none) -> CAP-US1206FAB; device fab_2:CAP-UNPOLARIZEDFAB -> fab_2:CAP-US1206FAB
Changed lines of the file:
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@@
 <part name="TH" library="thomasb9511" deviceset="SHT31-DIS" device=""/>
 <part name="CO2" library="T6713-6H" deviceset="T6713-6H" device=""/>
-<part name="FRAME1" library="frames" deviceset="A4L-LOC" device=""/>
+<part name="FRAME1" library="frames" deviceset="A4L-LOC" device="" value="C02"/>
 <part name="GND1" library="supply1" deviceset="GND" device=""/>
 <part name="GND2" library="supply1" deviceset="GND" device=""/>
@@
 <part name="R3" library="fab" deviceset="RES-US" device="1206FAB" value="10k"/>
 <part name="R4" library="fab" deviceset="RES-US" device="1206FAB" value="0"/>
-<part name="C1" library="fab_2" deviceset="CAP-UNPOLARIZED" device="FAB"/>
+<part name="C1" library="fab_2" deviceset="CAP-US" device="1206FAB" value=""/>
 <part name="GND3" library="supply1" deviceset="GND" device=""/>
 <part name="R5" library="fab" deviceset="RES-US" device="1206FAB" value="0"/>
@@
 <instance part="R3" gate="G$1" x="38.1" y="142.24" rot="MR0"/>
 <instance part="R4" gate="G$1" x="55.88" y="93.98"/>
-<instance part="C1" gate="&gt;NAME" x="22.86" y="152.4" rot="R180"/>
+<instance part="C1" gate="G$1" x="22.86" y="152.4" rot="R180"/>
 <instance part="GND3" gate="1" x="17.78" y="142.24"/>
 <instance part="R5" gate="G$1" x="55.88" y="104.14"/>
@@
 <wire x1="43.18" y1="152.4" x2="43.18" y2="147.32" width="0.1524" layer="91"/>
 <wire x1="43.18" y1="147.32" x2="45.72" y2="147.32" width="0.1524" layer="91"/>
-<pinref part="C1" gate="&gt;NAME" pin="1"/>
-<wire x1="27.94" y1="152.4" x2="30.48" y2="152.4" width="0.1524" layer="91"/>
+<pinref part="C1" gate="G$1" pin="1"/>
+<wire x1="25.4" y1="152.4" x2="30.48" y2="152.4" width="0.1524" layer="91"/>
 <junction x="43.18" y="152.4"/>
 <pinref part="R3" gate="G$1" pin="2"/>
@@
 <wire x1="60.96" y1="40.64" x2="60.96" y2="33.02" width="0.1524" layer="91"/>
 <pinref part="P+5" gate="VCC" pin="VCC"/>
+<junction x="60.96" y="40.64"/>
 </segment>
 <segment>
@@
 </segment>
 <segment>
-<pinref part="C1" gate="&gt;NAME" pin="2"/>
-<wire x1="20.32" y1="152.4" x2="17.78" y2="152.4" width="0.1524" layer="91"/>
+<pinref part="C1" gate="G$1" pin="2"/>
 <wire x1="17.78" y1="152.4" x2="17.78" y2="144.78" width="0.1524" layer="91"/>
 <pinref part="GND3" gate="1" pin="GND"/>
@@
 <wire x1="48.26" y1="99.06" x2="43.18" y2="99.06" width="0.1524" layer="91"/>
 <label x="43.18" y="99.06" size="1.778" layer="95" rot="R180" xref="yes"/>
+<junction x="48.26" y="99.06"/>
 </segment>
 </net>
