File: V.raspberryPi/Ecotron/EAGLE/PCB/board_0.2v.brd (EAGLE design)
At the start: 100 x 80 mm, 26 parts, among them J4 4P-2.0, J5 4P-2.0, J6 4P-2.0, U1 ADS1015, U4 PCA9546APW,112

Commit message: seedstudio finish
Parts:
- moved R8 138.1 mm to (98.3, 24.9), turned to 90 degrees
- moved R4 123.0 mm to (86.7, 40.7), turned to 90 degrees
- moved R5 120.8 mm to (74.3, 41.8), turned to 90 degrees
- moved R6 120.7 mm to (63.2, 42.6), turned to 90 degrees
- moved R9 117.1 mm to (54.3, 24.1), turned to 90 degrees
- moved R7 115.0 mm to (71.6, 23.8), turned to 90 degrees
- moved C3 66.7 mm to (8.40, 23.9), turned to 180 degrees
- moved R3 48.5 mm to (2.60, 18.8), turned to 270 degrees
- moved R2 41.4 mm to (15.1, 16.1)
- moved R1 38.8 mm to (15.2, 19.7)
- moved C2 35.1 mm to (2.80, 24.6), turned to 90 degrees
- moved C1 34.6 mm to (2.50, 30.5), turned to 270 degrees
- moved U4 3.36 mm to (21.6, 29.8), turned to 180 degrees
- moved U3 3.32 mm to (11.4, 29.6)
Changed lines of the file:
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@@
 <attribute name="PROD_ID" value="IC-12270" x="8" y="18.9" size="1.778" layer="27" rot="R270" display="off"/>
 </element>
-<element name="U3" library="adafruit" package="TSSOP20" value="" x="8.1" y="29.2"/>
+<element name="U3" library="adafruit" package="TSSOP20" value="" x="11.4" y="29.6"/>
 <element name="T1" library="fab_2" package="TO252" value="" x="88.6" y="15.3"/>
 <element name="T2" library="fab_2" package="TO252" value="" x="77" y="15.1"/>
@@
 <element name="J5" library="Seeed-OPL-Connector" package="HW4-2.0" value="4P-2.0" x="23.5" y="5.7"/>
 <element name="J6" library="Seeed-OPL-Connector" package="HW4-2.0" value="4P-2.0" x="36.5" y="5.7"/>
-<element name="U4" library="NXP_By_element14_Batch_1" package="SOP65P640X110-16N" value="PCA9546APW,112" x="24.7" y="28.5" rot="R90">
-<attribute name="OC_NEWARK" value="70R6610" x="24.7" y="28.5" size="1.778" layer="27" rot="R90" display="off"/>
-<attribute name="SUPPLIER" value="NXP" x="24.7" y="28.5" size="1.778" layer="27" rot="R90" display="off"/>
-<attribute name="OC_FARNELL" value="1831208" x="24.7" y="28.5" size="1.778" layer="27" rot="R90" display="off"/>
-<attribute name="MPN" value="PCA9546APW,112" x="24.7" y="28.5" size="1.778" layer="27" rot="R90" display="off"/>
-<attribute name="PACKAGE" value="TSSOP-16" x="24.7" y="28.5" size="1.778" layer="27" rot="R90" display="off"/>
+<element name="U4" library="NXP_By_element14_Batch_1" package="SOP65P640X110-16N" value="PCA9546APW,112" x="21.6" y="29.8" rot="R180">
+<attribute name="OC_NEWARK" value="70R6610" x="21.6" y="29.8" size="1.778" layer="27" rot="R180" display="off"/>
+<attribute name="SUPPLIER" value="NXP" x="21.6" y="29.8" size="1.778" layer="27" rot="R180" display="off"/>
+<attribute name="OC_FARNELL" value="1831208" x="21.6" y="29.8" size="1.778" layer="27" rot="R180" display="off"/>
+<attribute name="MPN" value="PCA9546APW,112" x="21.6" y="29.8" size="1.778" layer="27" rot="R180" display="off"/>
+<attribute name="PACKAGE" value="TSSOP-16" x="21.6" y="29.8" size="1.778" layer="27" rot="R180" display="off"/>
 </element>
-<element name="C1" library="fab" package="C1206FAB" value="CAP-US1206FAB" x="2.4" y="-4.1"/>
-<element name="C2" library="fab" package="C1206FAB" value="CAP-US1206FAB" x="2.4" y="-10.5"/>
-<element name="R1" library="fab" package="R1206FAB" value="" x="2.4" y="-16.9"/>
-<element name="R2" library="fab" package="R1206FAB" value="" x="2.4" y="-23.3"/>
-<element name="R3" library="fab" package="R1206FAB" value="" x="2.4" y="-29.7"/>
-<element name="C3" library="fab" package="C1206FAB" value="CAP-US1206FAB" x="2.4" y="-42.5"/>
-<element name="R4" library="fab" package="R1206FAB" value="" x="2.4" y="-48.9"/>
-<element name="R5" library="fab" package="R1206FAB" value="" x="2.4" y="-55.3"/>
-<element name="R6" library="fab" package="R1206FAB" value="" x="2.4" y="-61.7"/>
-<element name="R7" library="fab" package="R1206FAB" value="" x="2.4" y="-68.1"/>
-<element name="R8" library="fab" package="R1206FAB" value="" x="2.4" y="-74.5"/>
-<element name="R9" library="fab" package="R1206FAB" value="" x="2.4" y="-80.9"/>
+<element name="C1" library="fab" package="C1206FAB" value="CAP-US1206FAB" x="2.5" y="30.5" rot="R270"/>
+<element name="C2" library="fab" package="C1206FAB" value="CAP-US1206FAB" x="2.8" y="24.6" rot="R90"/>
+<element name="R1" library="fab" package="R1206FAB" value="" x="15.2" y="19.7"/>
+<element name="R2" library="fab" package="R1206FAB" value="" x="15.1" y="16.1"/>
+<element name="R3" library="fab" package="R1206FAB" value="" x="2.6" y="18.8" rot="R270"/>
+<element name="C3" library="fab" package="C1206FAB" value="CAP-US1206FAB" x="8.4" y="23.9" rot="R180"/>
+<element name="R4" library="fab" package="R1206FAB" value="" x="86.7" y="40.7" rot="R90"/>
+<element name="R5" library="fab" package="R1206FAB" value="" x="74.3" y="41.8" rot="R90"/>
+<element name="R6" library="fab" package="R1206FAB" value="" x="63.2" y="42.6" rot="R90"/>
+<element name="R7" library="fab" package="R1206FAB" value="" x="71.6" y="23.8" rot="R90"/>
+<element name="R8" library="fab" package="R1206FAB" value="" x="98.3" y="24.9" rot="R90"/>
+<element name="R9" library="fab" package="R1206FAB" value="" x="54.3" y="24.1" rot="R90"/>
 </elements>
 <signals>
@@
 <contactref element="C2" pad="2"/>
 <contactref element="C3" pad="2"/>
-<wire x1="26.986" y1="25.579" x2="31.15" y2="54.57" width="0" layer="19" extent="1-1"/>
-<wire x1="11.025" y1="32.1178" x2="26.986" y2="25.579" width="0" layer="19" extent="1-1"/>
-<wire x1="5.95" y1="18.9" x2="11.025" y2="32.1178" width="0" layer="19" extent="1-1"/>
+<wire x1="24.521" y1="32.086" x2="31.15" y2="54.57" width="0" layer="19" extent="1-1"/>
+<wire x1="14.325" y1="32.5178" x2="24.521" y2="32.086" width="0" layer="19" extent="1-1"/>
+<wire x1="5.95" y1="18.9" x2="14.325" y2="32.5178" width="0" layer="19" extent="1-1"/>
 <wire x1="13" y1="5.7" x2="5.95" y2="18.9" width="0" layer="19" extent="1-1"/>
-<wire x1="4.051" y1="-4.1" x2="13" y2="5.7" width="0" layer="19" extent="1-1"/>
-<wire x1="4.051" y1="-10.5" x2="4.051" y2="-4.1" width="0" layer="19" extent="1-1"/>
+<wire x1="2.5" y1="28.849" x2="13" y2="5.7" width="0" layer="19" extent="1-1"/>
+<wire x1="2.8" y1="26.251" x2="2.5" y2="28.849" width="0" layer="19" extent="1-1"/>
 <wire x1="26.5" y1="5.7" x2="13" y2="5.7" width="0" layer="19" extent="1-1"/>
 <wire x1="39.5" y1="5.7" x2="26.5" y2="5.7" width="0" layer="19" extent="1-1"/>
-<wire x1="4.051" y1="-42.5" x2="4.051" y2="-10.5" width="0" layer="19" extent="1-1"/>
+<wire x1="6.749" y1="23.9" x2="2.8" y2="26.251" width="0" layer="19" extent="1-1"/>
 </signal>
 <signal name="GPIO17">
@@
 <contactref element="U3" pad="19"/>
 <contactref element="C1" pad="1"/>
-<wire x1="0.749" y1="-4.1" x2="5.825" y2="32.1178" width="0" layer="19" extent="1-1"/>
+<wire x1="2.5" y1="32.151" x2="9.125" y2="32.5178" width="0" layer="19" extent="1-1"/>
 </signal>
 <signal name="N$27">
 <contactref element="U3" pad="2"/>
 <contactref element="C2" pad="1"/>
-<wire x1="0.749" y1="-10.5" x2="5.825" y2="26.2822" width="0" layer="19" extent="1-1"/>
+<wire x1="2.8" y1="22.949" x2="9.125" y2="26.6822" width="0" layer="19" extent="1-1"/>
 </signal>
 <signal name="N$24">
 <contactref element="U1" pad="8"/>
 <contactref element="C3" pad="1"/>
-<wire x1="10.05" y1="18.9" x2="0.749" y2="-42.5" width="0" layer="19" extent="1-1"/>
+<wire x1="10.05" y1="18.9" x2="10.051" y2="23.9" width="0" layer="19" extent="1-1"/>
 </signal>
 <signal name="N$29">
 <contactref element="U1" pad="10"/>
 <contactref element="R1" pad="1"/>
-<wire x1="0.749" y1="-16.9" x2="10.05" y2="19.9" width="0" layer="19" extent="1-1"/>
+<wire x1="13.549" y1="19.7" x2="10.05" y2="19.9" width="0" layer="19" extent="1-1"/>
 </signal>
 <signal name="N$31">
 <contactref element="U1" pad="9"/>
 <contactref element="R2" pad="1"/>
-<wire x1="0.749" y1="-23.3" x2="10.05" y2="19.4" width="0" layer="19" extent="1-1"/>
+<wire x1="13.449" y1="16.1" x2="10.05" y2="19.4" width="0" layer="19" extent="1-1"/>
 </signal>
 <signal name="N$32">
 <contactref element="R1" pad="2"/>
 <contactref element="R2" pad="2"/>
-<wire x1="4.051" y1="-16.9" x2="4.051" y2="-23.3" width="0" layer="19" extent="1-1"/>
+<wire x1="16.851" y1="19.7" x2="16.751" y2="16.1" width="0" layer="19" extent="1-1"/>
 </signal>
 <signal name="N$33">
 <contactref element="U1" pad="1"/>
 <contactref element="R3" pad="1"/>
-<wire x1="5.95" y1="19.9" x2="0.749" y2="-29.7" width="0" layer="19" extent="1-1"/>
+<wire x1="5.95" y1="19.9" x2="2.6" y2="20.451" width="0" layer="19" extent="1-1"/>
 </signal>
 <signal name="N$34">
@@
 <contactref element="R7" pad="1"/>
 <contactref element="T2" pad="1"/>
-<wire x1="0.749" y1="-68.1" x2="74.72" y2="10.3" width="0" layer="19" extent="1-1"/>
+<wire x1="71.6" y1="22.149" x2="74.72" y2="10.3" width="0" layer="19" extent="1-1"/>
 </signal>
 <signal name="N$64">
 <contactref element="T5" pad="1"/>
 <contactref element="R6" pad="1"/>
-<wire x1="0.749" y1="-61.7" x2="62.42" y2="27.2" width="0" layer="19" extent="1-1"/>
+<wire x1="63.2" y1="40.949" x2="62.42" y2="27.2" width="0" layer="19" extent="1-1"/>
 </signal>
 <signal name="N$65">
 <contactref element="R8" pad="1"/>
 <contactref element="T1" pad="1"/>
-<wire x1="0.749" y1="-74.5" x2="86.32" y2="10.5" width="0" layer="19" extent="1-1"/>
+<wire x1="98.3" y1="23.249" x2="86.32" y2="10.5" width="0" layer="19" extent="1-1"/>
 </signal>
 <signal name="N$66">
 <contactref element="T4" pad="1"/>
 <contactref element="R9" pad="1"/>
-<wire x1="62.22" y1="10.1" x2="0.749" y2="-80.9" width="0" layer="19" extent="1-1"/>
+<wire x1="62.22" y1="10.1" x2="54.3" y2="22.449" width="0" layer="19" extent="1-1"/>
 </signal>
 <signal name="N$67">
 <contactref element="R5" pad="1"/>
 <contactref element="T3" pad="1"/>
-<wire x1="0.749" y1="-55.3" x2="74.72" y2="26.9" width="0" layer="19" extent="1-1"/>
+<wire x1="74.3" y1="40.149" x2="74.72" y2="26.9" width="0" layer="19" extent="1-1"/>
 </signal>
 <signal name="N$68">
 <contactref element="R4" pad="1"/>
 <contactref element="T6" pad="1"/>
-<wire x1="0.749" y1="-48.9" x2="86.12" y2="27" width="0" layer="19" extent="1-1"/>
+<wire x1="86.7" y1="39.049" x2="86.12" y2="27" width="0" layer="19" extent="1-1"/>
 </signal>
 <signal name="N$69">
