File: V.raspberryPi/Ecotron/EAGLE/PCB/board_0.4v.sch (EAGLE design)
At the start: 16 parts, among them J4 4P-2.0, J5 4P-2.0, J6 4P-2.0, U1 ADS1015, U4 PCA9546APW,112

Commit message: add
Parts:
- removed T5: (no value), fab_2:NMOSFETTO252
- removed U$1: RPI-ZERO, RPI-Zero:RPI-ZERO
- added C3: 1uf, Seeed-OPL-Capacitor:CERAMIC-1UF-25V-10%-X7R(0805)
- added J1, J2, J3: 1X2-3.5MM, adafruit:1X2-3.5MM
- added JP2: (no value), adafruit:PINHD-1X8BIG
- added JP3: (no value), pinhead:PINHD-1X4
- added JP4, JP5: (no value), adafruit:PINHD-2X4
- added R1, R2, R3, R4, R5, R6, R7: 10K, Seeed-OPL-Resistor:SMD-RES-10K-1%-1/8W(0805)
- added U$2, U$3, U$4: SOLDER_JUMPER, fab:SOLDER_JUMPER
- added U2: (no value), adafruit:PCA9685
- C1, C2: value CAP-US1206FAB -> 1uf; device fab:CAP-US1206FAB -> Seeed-OPL-Capacitor:CERAMIC-1UF-25V-10%-X7R(0805)
- T4, T6: value (none) -> MOSFET-N; device fab_2:NMOSFETTO252 -> Seeed-OPL-Transistor:MOSFET-N
Connections:
- removed net GND_2: JP1.9
- removed net N$14: U3.OE
- removed net N$27: C2.1, U3.VCCA
- removed net SDL: JP1.5
- new net 12V: J2.1, T1.D, T2.D, T3.D, T4.D, T6.D
- new net 3,3_1V: U4.VDD
- new net A0+: JP3.4, U1.AIN0
- new net A0-: JP3.3, U1.AIN1
- new net A1+: JP3.1, U1.AIN2
- new net A1-: JP3.2, U1.AIN3
- new net ADDR_AD: U$3.1, U$4.1, U1.ADDR
- new net N$10: R6.1, T4.G
- new net N$11: R7.1, T2.G
- new net N$12: R5.1, T3.G
- new net N$6: R3.1, T6.G
- new net N$7: J4.2
- new net N$8: J4.1
- new net N$9: R4.1, T1.G
- new net OE: U$2.1, U3.OE
- new net SC0: J5.1, U4.SC0
- new net SC1: J6.1, U4.SC1
- new net SC2: U4.SC2
- new net SC3: U4.SC3
- new net SCL: JP1.5, R2.2, U1.SCL, U4.SCL
- new net SD0: J5.2, U4.SD0
- new net SD1: J6.2, U4.SD1
- new net SD2: U4.SD2
- new net SD3: U4.SD3
- new net VCC: J4.3, J5.3, J6.3
- net 3,3V: now also C3.1, R1.1, R2.1, U$3.2, U1.VDD
- net 3,3V_1: now also C2.1, U$2.2, U3.VCCA
- net GND: now also C3.2, J2.2, JP1.9, T1.S, T2.S, T3.S, T4.S, T6.S, U$4.2, U1.ALERT/RDY, U4.A0, U4.A1, U4.A2
- net GPIO10: now also U3.A8; no longer U3.A1
- net GPIO11: now also U3.A6; no longer U3.A3
- net GPIO13: now also U3.A4; no longer U3.A5
- net GPIO14: now also R3.2
- net GPIO15: now also R6.2
- net GPIO18: now also R5.2
- net GPIO19: now also U3.A3; no longer U3.A6
- net GPIO21: now also U3.A1
- net GPIO23: now also R7.2; no longer U3.A7
- net GPIO26: now also U3.A2; no longer U3.A8
- net GPIO6: now also U3.A5; no longer U3.A4
- net GPIO8: now also R4.2
- net GPIO9: now also U3.A7; no longer U3.A2
- net N$15: now also JP2.8
- net N$16: now also JP2.7
- net N$17: now also JP2.6
- net N$18: now also JP2.5
- net N$19: now also JP2.4
- net N$20: now also JP2.3
- net N$21: now also JP2.2
- net N$22: now also JP2.1
- net SDA: now also R1.2, U1.SDA, U4.SDA
Other:
- moved on the sheet: T1, T2, T3
