File: V.raspberryPi/Ecotron/EAGLE/PCB/board_0.6v.sch (EAGLE design)
At the start: 16 parts, among them J4 4P-2.0, J5 4P-2.0, J6 4P-2.0, U1 ADS1015, U4 PCA9546APW,112

Commit message: add
Parts:
- removed T3, T5: (no value), fab_2:NMOSFETTO252
- removed U$1: RPI-ZERO, RPI-Zero:RPI-ZERO
- added C3: 1uf, Seeed-OPL-Capacitor:CERAMIC-1UF-25V-10%-X7R(0805)
- added J1, J2, J3: 1X2-3.5MM, adafruit:1X2-3.5MM
- added JP2, JP4, JP5: (no value), adafruit:PINHD-2X4
- added JP3: (no value), pinhead:PINHD-1X4
- added JP6: (no value), pinhead:PINHD-2X2
- added R1, R2, R3, R4, R6, R7: 10K, Seeed-OPL-Resistor:SMD-RES-10K-1%-1/8W(0805)
- added U$3, U$4: SOLDER_JUMPER, fab:SOLDER_JUMPER
- added U2: (no value), adafruit:PCA9685
- C1, C2: value CAP-US1206FAB -> 1uf; device fab:CAP-US1206FAB -> Seeed-OPL-Capacitor:CERAMIC-1UF-25V-10%-X7R(0805)
- T4, T6: value (none) -> MOSFET-N; device fab_2:NMOSFETTO252 -> Seeed-OPL-Transistor:MOSFET-N
Connections:
- removed net GND_2: JP1.9
- removed net N$18: U3.B5
- removed net N$19: U3.B4
- removed net N$20: U3.B3
- removed net N$21: U3.B2
- removed net SDL: JP1.5
- new net 12V: J2.1, T1.D, T2.D, T4.D, T6.D
- new net 3,3_1V: U4.VDD
- new net A0+: JP3.4, U1.AIN0
- new net A0-: JP3.3, U1.AIN1
- new net A1+: JP3.1, U1.AIN2
- new net A1-: JP3.2, U1.AIN3
- new net ADDR_AD: U$3.1, U$4.1, U1.ADDR
- new net B1: JP5.7, U3.B1
- new net B2: JP5.8, U3.B2
- new net B3: JP5.5, U3.B3
- new net B4: JP5.6, U3.B4
- new net B5: JP5.3, U3.B5
- new net B6: JP5.4, U3.B6
- new net B7: JP5.1, U3.B7
- new net B8: JP5.2, U3.B8
- new net N$10: R6.1, T4.G
- new net N$11: R7.1, T2.G
- new net N$13: JP2.1
- new net N$24: U2.PWM9
- new net N$28: U2.PWM11
- new net N$29: U2.PWM12
- new net N$31: U2.PWM13
- new net N$32: U2.PWM14
- new net N$33: U2.PWM15
- new net N$6: R3.1, T6.G
- new net N$7: J4.2
- new net N$8: J4.1
- new net N$9: R4.1, T1.G
- new net PWM0: JP4.2, U2.PWM0
- new net PWM1: JP4.1, U2.PWM1
- new net PWM2: JP4.4, U2.PWM2
- new net PWM3: JP4.3, U2.PWM3
- new net PWM4: JP4.6, U2.PWM4
- new net PWM5: JP4.5, U2.PWM5
- new net PWM6: JP4.8, U2.PWM6
- new net PWM7: JP4.7, U2.PWM7
- new net SC0: J5.1, U4.SC0
- new net SC1: J6.1, U4.SC1
- new net SC2: U4.SC2
- new net SC3: U4.SC3
- new net SCL: JP1.5, R2.2, U1.SCL, U2.SCL, U4.SCL
- new net SD0: J5.2, U4.SD0
- new net SD1: J6.2, U4.SD1
- new net SD2: U4.SD2
- new net SD3: U4.SD3
- new net VCC: J4.3, J5.3, J6.3
- net 3,3V: now also C3.1, R1.1, R2.1, U$3.2, U1.VDD, U2.A0, U2.A2, U2.A4, U2.VDD
- net 3,3V_1: now also C2.1, U3.OE, U3.VCCA
- net GND: now also C3.2, J2.2, JP1.9, T1.S, T2.S, T4.S, T6.S, U$4.2, U1.ALERT/RDY, U2.A1, U2.A3, U2.A5, U2.EXTCLK, U2.GND, U4.A0, U4.A1, U4.A2
- net GPIO10: now also U3.A8; no longer U3.A1
- net GPIO11: now also U3.A6; no longer U3.A3
- net GPIO13: now also U3.A4; no longer U3.A5
- net GPIO14: now also R3.2
- net GPIO15: now also R6.2
- net GPIO19: now also U3.A3; no longer U3.A6
- net GPIO21: now also U3.A1
- net GPIO23: now also R7.2; no longer U3.A7
- net GPIO26: now also U3.A2; no longer U3.A8
- net GPIO6: now also U3.A5; no longer U3.A4
- net GPIO8: now also R4.2
- net GPIO9: now also U3.A7; no longer U3.A2
- net N$14: now also JP2.3; no longer U3.OE
- net N$15: now also JP2.5; no longer U3.B8
- net N$16: now also U2.#OE; no longer U3.B7
- net N$17: now also JP2.7; no longer U3.B6
- net N$22: now also U2.PWM8; no longer U3.B1
- net N$27: now also U2.PWM10; no longer C2.1, U3.VCCA
- net SDA: now also R1.2, U1.SDA, U2.SDA, U4.SDA
Other:
- moved on the sheet: T1, T2
