File: V.raspberryPi/Ecotron/EAGLE/PCB/board_0.8v.sch (EAGLE design)
At the start: 35 parts, among them J1 1X2-3.5MM, J2 1X2-3.5MM, J3 1X2-3.5MM, J4 4P-2.0, J5 4P-2.0, J6 4P-2.0, J7 4P-2.0, T1 T1, T2 T2, T4 MOSFET-N, T6 MOSFET-N, U1 ADS1015, U2 PCA9685, U3 TXB0108, U4 PCA9546APW,112

Commit message: update board
Parts:
- removed J1, J2, J3: 1X2-3.5MM, adafruit:1X2-3.5MM
- removed J4, J5, J6, J7: 4P-2.0, Seeed-OPL-Connector:GROVE-CONNECTOR-DIP(4P-2.0)
- removed JP4: PWM, adafruit:PINHD-2X4
- removed JP7: ADC, pinhead:PINHD-2X2
- removed SJ1: ADDR, jumper:SJ2W
- removed U$1: 10K, Seeed-OPL-Resistor:SMD-RES-10K-1%-1/8W(0805)
- added ADC, ADC-1, MOSFET-1, PWD, PWD1: (no value), pinhead:PINHD-2X2
- added C5: 100nf, Seeed-OPL-Capacitor:CERAMIC-100NF-50V-10%-X7R(0805)
- added I2C-0, I2C-1, I2C-2, I2C-3: 4P-2.0, Seeed-OPL-Connector:GROVE-CONNECTOR-DIP(4P-2.0)
- added INPUT: 1X2-3.5MM, adafruit:1X2-3.5MM
- added PWM: PWM, adafruit:PINHD-2X4
- added R8: 10K, Seeed-OPL-Resistor:SMD-RES-10K-1%-1/8W(0805)
- added RPI: GPIO, adafruit:PINHD-2X20
- added U5: ADS1015, SparkFun-IC-Conversion:ADS1015
- C3: value 0.1uf -> 100nf; device Seeed-OPL-Capacitor:CERAMIC-1UF-25V-10%-X7R(0805) -> Seeed-OPL-Capacitor:CERAMIC-100NF-50V-10%-X7R(0805)
- JP1: value GPIO -> JUMPER-SMT_3_NO_SILK; device adafruit:PINHD-2X20 -> SparkFun-Jumpers:JUMPER-SMT_3_NO_SILK
- JP2: value PWM -> JUMPER-SMT_3_NO_SILK; device adafruit:PINHD-2X4 -> SparkFun-Jumpers:JUMPER-SMT_3_NO_SILK
- renumbered JP5 to OUTPUT, JP6 to MOSFET
Connections:
- removed net ADDR_AD: SJ1.2, U1.ADDR
- removed net VCC: J4.3, J5.3, J6.3, J7.3
- new net A0+_1: ADC-1.3, U5.AIN0
- new net A0-_1: ADC-1.1, U5.AIN1
- new net A1+_1: ADC-1.2, U5.AIN2
- new net A1-_1: ADC-1.4, U5.AIN3
- new net N$13: C5.1, U1.VDD
- new net N$8: C3.1, U5.VDD
- new net VCC_I2C_1: I2C-0.3, I2C-1.3, JP1.2
- new net VCC_I2C_2: I2C-2.3, I2C-3.3, JP2.2
- net 12V: now also INPUT.1, PWD1.1, PWD1.3; no longer J2.1
- net 3,3V: now also C3.2, C5.2, JP2.3, PWD.1, RPI.1, U1.ADDR; no longer C3.1, SJ1.1, U1.VDD
- net 3,3V_1: now also RPI.17; no longer JP1.17
- net 5V: now also JP1.3, JP2.1, PWD.3, RPI.2; no longer JP1.2
- net A0+: now also ADC.3; no longer JP7.1
- net A0-: now also ADC.1; no longer JP7.2
- net A1+: now also ADC.2; no longer JP7.4
- net A1-: now also ADC.4; no longer JP7.3
- net CLK: now also RPI.7; no longer JP1.7
- net GND: now also I2C-0.4, I2C-1.4, I2C-2.4, I2C-3.4, INPUT.2, MOSFET-1.3, MOSFET-1.4, PWD.2, PWD.4, PWD1.2, PWD1.4, R8.1, RPI.14, RPI.25, RPI.30, RPI.39, RPI.6, RPI.9, U5.ADDR, U5.ALERT/RDY, U5.VSS; no longer C3.2, J1.2, J2.2, J3.2, J4.4, J5.4, J6.4, J7.4, JP1.14, JP1.25, JP1.30, JP1.39, JP1.6, JP1.9, SJ1.3, U$1.1
- net GND_3: now also RPI.20; no longer JP1.20
- net GND_6: now also RPI.34; no longer JP1.34
- net GPIO10: now also RPI.19; no longer JP1.19
- net GPIO11: now also RPI.23; no longer JP1.23
- net GPIO12: now also RPI.32; no longer JP1.32
- net GPIO13: now also RPI.33; no longer JP1.33
- net GPIO14: now also RPI.8; no longer JP1.8
- net GPIO15: now also RPI.10; no longer JP1.10
- net GPIO16: now also RPI.36; no longer JP1.36
- net GPIO17: now also RPI.11; no longer JP1.11
- net GPIO18: now also RPI.12; no longer JP1.12
- net GPIO19: now also RPI.35; no longer JP1.35
- net GPIO20: now also RPI.38; no longer JP1.38
- net GPIO21: now also RPI.40; no longer JP1.40
- net GPIO22: now also RPI.15; no longer JP1.15
- net GPIO23: now also RPI.16; no longer JP1.16
- net GPIO26: now also RPI.37; no longer JP1.37
- net GPIO27: now also RPI.13; no longer JP1.13
- net GPIO5: now also RPI.29; no longer JP1.29
- net GPIO6: now also RPI.31; no longer JP1.31
- net GPIO7: now also RPI.26; no longer JP1.26
- net GPIO8: now also RPI.24; no longer JP1.24
- net GPIO9: now also RPI.21; no longer JP1.21
- net MOSFET_3: now also MOSFET-1.2; no longer J1.1
- net MOSFET_4: now also MOSFET-1.1; no longer J3.1
- net N$16: now also R8.2; no longer U$1.2
- net N$23: now also RPI.18; no longer JP1.18
- net N$25: now also RPI.22; no longer JP1.22
- net N$30: now also RPI.27; no longer JP1.27
- net N$38: now also RPI.28; no longer JP1.28
- net N$5: now also RPI.4; no longer JP1.4
- net PWM0: now also PWM.2; no longer JP4.2
- net PWM1: now also PWM.1; no longer JP4.1
- net PWM10: no longer JP2.3
- net PWM11: no longer JP2.4
- net PWM12: no longer JP2.5
- net PWM13: no longer JP2.6
- net PWM14: no longer JP2.7
- net PWM15: no longer JP2.8
- net PWM2: now also PWM.4; no longer JP4.4
- net PWM3: now also PWM.3; no longer JP4.3
- net PWM4: now also PWM.6; no longer JP4.6
- net PWM5: now also PWM.5; no longer JP4.5
- net PWM6: now also PWM.8; no longer JP4.8
- net PWM7: now also PWM.7; no longer JP4.7
- net PWM8: no longer JP2.1
- net PWM9: no longer JP2.2
- net SC0: now also I2C-0.1; no longer J5.1
- net SC1: now also I2C-1.1; no longer J6.1
- net SC2: now also I2C-2.1; no longer J4.1
- net SC3: now also I2C-3.1; no longer J7.1
- net SCL: now also RPI.5, U5.SCL; no longer JP1.5
- net SD0: now also I2C-0.2; no longer J5.2
- net SD1: now also I2C-1.2; no longer J6.2
- net SD2: now also I2C-2.2; no longer J4.2
- net SD3: now also I2C-3.2; no longer J7.2
- net SDA: now also RPI.3, U5.SDA; no longer JP1.3
Other:
- note added: "AD 12Bits / 2"
- note added: "HAT Biotech Version 0.8"
- note removed: "CAPACITORES A LA SALIDA DEL ADC"
- note removed: "HAT Biotech Version 1.0"
- moved on the sheet: C3, C4, C6, R1, R2, R5, U1, U2, U4
